Commit message: spawnando robô só que com problemas

File: urdf/robozinho.urdf.xacro (robot description, xacro)
@@ -28,13 +28,13 @@
   <link name="base_link">
     <visual>
-      <origin xyz="0 0 3.14" rpy="0 0 3.14"/>
+      <origin xyz="0 0 0" rpy="0 0 3.14"/>
       <geometry>
-        <mesh filename="package://rocket/meshes/EST_estrutura_m3.dae" />
+        <mesh filename="file:////home/gabs/workspace/src/rocket/meshes/EST_estrutura_m3.dae" />
       </geometry>
     </visual>
     <collision>
-        <origin rpy="0  0  3.14" xyz="0  0  0.0118" />
+        <origin rpy="0  0  3.14" xyz="0  0  0" />
         <geometry>
-            <mesh filename="package://meshes/EST_estrutura_m3.dae" scale="1 1 1" />
+            <mesh filename="file:////home/gabs/workspace/src/rocket/meshes/EST_estrutura_m3.dae" scale="1 1 1" />
         </geometry>
     </collision>
@@ -53,5 +53,5 @@
         <origin xyz="0 0 0" rpy="0 0 0"/>
         <geometry>
-            <mesh filename="package://rocket/meshes/M_rodatrativa.dae" scale="1 1 1"/>
+            <mesh filename="file:////home/gabs/workspace/src/rocket/meshes/M_rodatrativa.dae" scale="1 1 1"/>
         </geometry>
       </visual>
@@ -59,5 +59,5 @@
         <origin xyz="0 0 0" rpy="0 0 0"/>
         <geometry>
-          <mesh filename="package://meshes/M_rodatrativa.dae" scale="1 1 1"/>
+          <mesh filename="file:////home/gabs/workspace/src/rocket/meshes/M_rodatrativa.dae" scale="1 1 1"/>
         </geometry>
       </collision>
@@ -78,5 +78,5 @@
         </joint>
    </xacro:macro>
-    <xacro:traction_wheel prefix="left_wheel" pos_X="-0.214" pos_Y="0" pos_Z="0.0507" pos_r="0" pos_p="1.57" pos_y="0" />
-    <xacro:traction_wheel prefix="right_wheel" pos_X="0.193" pos_Y="0" pos_Z="0.0507" pos_r="0" pos_p="1.57" pos_y="0" />
+  <xacro:wheel prefix="left_wheel" pos_X="-0.214" pos_Y="0" pos_Z="0.0507" pos_r="0" pos_p="1.57" pos_y="0" />
+  <xacro:wheel prefix="right_wheel" pos_X="0.193" pos_Y="0" pos_Z="0.0507" pos_r="0" pos_p="1.57" pos_y="0" />
 </robot>

Commit message: Rodas ajeitadas mas faltando colisão

File: urdf/robozinho.urdf.xacro (robot description, xacro)
@@ -3,10 +3,10 @@
   <!-- ****************** ROBOT CONSTANTS *******************************  -->
   <!-- Define the size of the robot's main chassis in meters -->
-  <xacro:property name="base_width" value="0.58"/>
-  <xacro:property name="base_length" value="0.85"/>
-  <xacro:property name="base_height" value="0.20"/>
+  <xacro:property name="base_width" value="0.557"/>
+  <xacro:property name="base_length" value="0.617"/>
+  <xacro:property name="base_height" value="0.182"/>
   <!-- Define the shape of the robot's two back wheels in meters -->
-  <xacro:property name="wheel_radius" value="0.14"/>
-  <xacro:property name="wheel_width" value="0.04"/>
+  <xacro:property name="wheel_radius" value="0.07"/>
+  <xacro:property name="wheel_width" value="0.03"/>
   <!-- x-axis points forward, y-axis points to left, z-axis points upwards -->
   <!-- Define the gap between the wheel and chassis along y-axis in meters -->
@@ -16,48 +16,45 @@
   <!-- Position the wheels along the x-axis -->
   <xacro:property name="wheel_xoff" value="0.221"/>
-  <!-- ****************** ROBOT BASE FOOTPRINT ***************************  -->
-  <!-- Define the center of the main robot chassis projected on the ground -->
-  <link name="base_footprint"/>
-  <!-- The base footprint of the robot is located underneath the chassis -->
-  <joint name="base_joint" type="fixed">
-    <parent link="base_footprint"/>
-    <child link="base_link" />
-    <origin xyz="0.0 0.0 0.0118" rpy="0 0 3.14"/>
-  </joint>
   <!-- ********************** ROBOT BASE *********************************  -->
   <link name="base_link">
-    <visual>
-      <origin xyz="0 0 0" rpy="0 0 3.14"/>
-      <geometry>
-        <mesh filename="file:////home/gabs/workspace/src/rocket/meshes/EST_estrutura_m3.dae" />
-      </geometry>
-    </visual>
-    <collision>
-        <origin rpy="0  0  3.14" xyz="0  0  0" />
+    </link>
+    <joint name="base_joint" type="fixed">
+      <parent link="base_link"/>
+      <child link="chassis" />
+      <origin xyz="0.0 0.0 0.0118" rpy="0 0 3.14"/>
+    </joint>
+    <link name="chassis">
+      <visual>
+        <origin xyz="0  0  0" rpy="0 0 0"/>
         <geometry>
-            <mesh filename="file:////home/gabs/workspace/src/rocket/meshes/EST_estrutura_m3.dae" scale="1 1 1" />
+          <mesh filename="file:////home/renata_a/workspace/src/rocket/meshes/EST_estrutura_m3.dae" />
         </geometry>
-    </collision>
-    <inertial>
-         <origin xyz="0  0  0.0118" rpy="0  0  3.14"/>
-         <mass value="2.4"/>
-         <inertia ixx="0.019995" ixy="0.0" ixz="0.0"
-               iyy="0.019995" iyz="0.0"
-               izz="0.03675" />
-    </inertial>
-  </link>
+      </visual>
+      <collision>
+          <origin rpy="0  0  0" xyz="0  0  0" />
+          <geometry>
+              <box size="${base_length} ${base_width} ${base_height}"/>
+          </geometry>
+      </collision>
+      <inertial>
+          <origin xyz="0  0  0.0118" rpy="0  0  3.14"/>
+          <mass value="2.4"/>
+          <inertia ixx="0.019995" ixy="0.0" ixz="0.0"
+                iyy="0.019995" iyz="0.0"
+                izz="0.03675" />
+      </inertial>
+    </link>
   <!-- *********************** DRIVE WHEELS ******************************  -->
-  <xacro:macro name="wheel" params="prefix pos_X pos_Y pos_Z pos_r pos_p pos_y">
-    <link name="${prefix}">
-      <visual name="${prefix}_visual">
+    <link name="left_wheel">
+      <visual name="left_wheel_visual">
         <origin xyz="0 0 0" rpy="0 0 0"/>
         <geometry>
-            <mesh filename="file:////home/gabs/workspace/src/rocket/meshes/M_rodatrativa.dae" scale="1 1 1"/>
+            <mesh filename="file:////home/renata_a/workspace/src/rocket/meshes/M_rodatrativa.dae" scale="1 1 1"/>
         </geometry>
       </visual>
-      <collision name="${prefix}_collision">
-        <origin xyz="0 0 0" rpy="0 0 0"/>
+      <collision name="left_wheel_collision">
+        <origin xyz="0 0 0" rpy="0 0 1.57"/>
         <geometry>
-          <mesh filename="file:////home/gabs/workspace/src/rocket/meshes/M_rodatrativa.dae" scale="1 1 1"/>
+          <cylinder length="${wheel_width}" radius="${wheel_radius}"/>
         </geometry>
       </collision>
@@ -70,13 +67,65 @@
       </inertial>
     </link>
-    <joint name="joint_${prefix}" type="revolute">
-            <parent link="base_link" />
-            <child link="${prefix}" />
-            <origin rpy="${pos_r} ${pos_p} ${pos_y}" xyz="${pos_X} ${pos_Y} ${pos_Z}" />
-            <axis xyz="0 0 1" />
-            <limit effort="-1.0" lower="-1e+16" upper="1e+16" velocity="-1.0" />
-        </joint>
-   </xacro:macro>
-  <xacro:wheel prefix="left_wheel" pos_X="-0.214" pos_Y="0" pos_Z="0.0507" pos_r="0" pos_p="1.57" pos_y="0" />
-  <xacro:wheel prefix="right_wheel" pos_X="0.193" pos_Y="0" pos_Z="0.0507" pos_r="0" pos_p="1.57" pos_y="0" />
+    <joint name="joint_left_wheel" type="revolute">
+            <parent link="chassis" />
+            <child link="left_wheel" />
+            <origin rpy="0 0 1.57" xyz="-0.098795 -0.296755 -0.09915" />
+            <axis rpy="0 0 0" xyz="0 1 0"/>
+            <limit effort="10000" velocity="1000"/>
+    </joint>
+    <link name="right_wheel">
+      <visual name="right_wheel_visual">
+        <origin xyz="0 0 0" rpy="0 0 0"/>
+        <geometry>
+            <mesh filename="file:////home/renata_a/workspace/src/rocket/meshes/M_rodatrativa.dae" scale="1 1 1"/>
+        </geometry>
+      </visual>
+      <collision name="right_wheel_collision">
+        <origin xyz="0 0 0" rpy="0 0 1.57"/>
+        <geometry>
+          <cylinder length="${wheel_width}" radius="${wheel_radius}"/>
+        </geometry>
+      </collision>
+      <inertial>
+        <mass value="1" />
+        <origin rpy="0 0 0" xyz="0 0 0" />
+        <inertia ixx="0.001" ixy="0.0" ixz="0.0"
+                iyy="0.001" iyz="0.0"
+                izz="0.001" />
+      </inertial>
+    </link>
+    <joint name="joint_right_wheel" type="revolute">
+            <parent link="chassis" />
+            <child link="right_wheel" />
+            <origin rpy="0 0 1.57" xyz="-0.098795 0.296395 -0.09915" />
+            <axis rpy="0 0 0" xyz="0 1 0"/>
+            <limit effort="10000" velocity="1000"/>
+    </joint>
+  <!-- *********************** TRAY ******************************  -->
+  <link name="tray">
+      <visual name="tray_visual">
+        <origin xyz="0 0 0.0118" rpy="0 0 0"/>
+        <geometry>
+            <mesh filename="file:////home/renata_a/workspace/src/rocket/meshes/ELV_conjuntocompleto.dae" scale="1 1 1"/>
+        </geometry>
+      </visual>
+      <collision name="tray_collision">
+        <origin xyz="0 0 0" rpy="0 0 0"/>
+        <geometry>
+          <mesh filename="file:////home/renata_a/workspace/src/rocket/meshes/ELV_conjuntocompleto.dae" scale="1 1 1"/>
+        </geometry>
+      </collision>
+      <inertial>
+        <mass value="0.5" />
+        <origin rpy="0 0 0" xyz="0 0 0" />
+        <inertia ixx="0.0" ixy="0.0" ixz="0.0"
+                iyy="0.0" iyz="0.0"
+                izz="0.0" />
+      </inertial>
+  </link>
+  <joint name="joint_tray" type="fixed">
+            <parent link="chassis" />
+            <child link="tray" />
+            <origin rpy="0 0 0" xyz="0 0 0" />
+    </joint>
 </robot>

Commit message: sdfg

File: urdf/robozinho.urdf.xacro (robot description, xacro)
@@ -28,5 +28,5 @@
         <origin xyz="0  0  0" rpy="0 0 0"/>
         <geometry>
-          <mesh filename="file:////home/renata_a/workspace/src/rocket/meshes/EST_estrutura_m3.dae" />
+          <mesh filename="file:///$(find rocket)/meshes/EST_estrutura_m3.dae" />
         </geometry>
       </visual>
@@ -50,5 +50,5 @@
         <origin xyz="0 0 0" rpy="0 0 0"/>
         <geometry>
-            <mesh filename="file:////home/renata_a/workspace/src/rocket/meshes/M_rodatrativa.dae" scale="1 1 1"/>
+            <mesh filename="file:///$(find rocket)/meshes/M_rodatrativa.dae" scale="1 1 1"/>
         </geometry>
       </visual>
@@ -78,5 +78,5 @@
         <origin xyz="0 0 0" rpy="0 0 0"/>
         <geometry>
-            <mesh filename="file:////home/renata_a/workspace/src/rocket/meshes/M_rodatrativa.dae" scale="1 1 1"/>
+            <mesh filename="file:///$(find rocket)/meshes/M_rodatrativa.dae" scale="1 1 1"/>
         </geometry>
       </visual>
@@ -107,5 +107,5 @@
         <origin xyz="0 0 0.0118" rpy="0 0 0"/>
         <geometry>
-            <mesh filename="file:////home/renata_a/workspace/src/rocket/meshes/ELV_conjuntocompleto.dae" scale="1 1 1"/>
+            <mesh filename="file:///$(find rocket)/meshes/ELV_conjuntocompleto.dae" scale="1 1 1"/>
         </geometry>
       </visual>
@@ -113,5 +113,5 @@
         <origin xyz="0 0 0" rpy="0 0 0"/>
         <geometry>
-          <mesh filename="file:////home/renata_a/workspace/src/rocket/meshes/ELV_conjuntocompleto.dae" scale="1 1 1"/>
+          <mesh filename="file:///$(find rocket)/meshes/ELV_conjuntocompleto.dae" scale="1 1 1"/>
         </geometry>
       </collision>

Commit message: Ajeitei as colisões básicas

File: urdf/robozinho.urdf.xacro (robot description, xacro)
@@ -5,15 +5,11 @@
   <xacro:property name="base_width" value="0.557"/>
   <xacro:property name="base_length" value="0.617"/>
-  <xacro:property name="base_height" value="0.182"/>
-  <!-- Define the shape of the robot's two back wheels in meters -->
+  <xacro:property name="base_height" value="0.1305"/>
+  <!-- Define the shape of the robot's two wheels in meters -->
   <xacro:property name="wheel_radius" value="0.07"/>
   <xacro:property name="wheel_width" value="0.03"/>
-  <!-- x-axis points forward, y-axis points to left, z-axis points upwards -->
-  <!-- Define the gap between the wheel and chassis along y-axis in meters -->
-  <xacro:property name="wheel_ygap" value="0.035"/>
-  <!-- Position the wheels along the z-axis -->
-  <xacro:property name="wheel_zoff" value="0.05"/>
-  <!-- Position the wheels along the x-axis -->
-  <xacro:property name="wheel_xoff" value="0.221"/>
+  <!-- Define the shape of the robot's tray in meters -->
+  <xacro:property name="tray_radius" value="0.2"/>
+  <xacro:property name="tray_width" value="0.041"/>
   <!-- ********************** ROBOT BASE *********************************  -->
   <link name="base_link">
@@ -28,9 +24,9 @@
         <origin xyz="0  0  0" rpy="0 0 0"/>
         <geometry>
-          <mesh filename="file:///$(find rocket)/meshes/EST_estrutura_m3.dae" />
+          <mesh filename="file:////home/renata_a/workspace/src/rocket/meshes/EST_estrutura_m3.dae" />
         </geometry>
       </visual>
       <collision>
-          <origin rpy="0  0  0" xyz="0  0  0" />
+          <origin rpy="0  0  0" xyz="0  0  -0.0118" />
           <geometry>
               <box size="${base_length} ${base_width} ${base_height}"/>
@@ -50,9 +46,9 @@
         <origin xyz="0 0 0" rpy="0 0 0"/>
         <geometry>
-            <mesh filename="file:///$(find rocket)/meshes/M_rodatrativa.dae" scale="1 1 1"/>
+            <mesh filename="file:////home/renata_a/workspace/src/rocket/meshes/M_rodatrativa.dae" scale="1 1 1"/>
         </geometry>
       </visual>
       <collision name="left_wheel_collision">
-        <origin xyz="0 0 0" rpy="0 0 1.57"/>
+        <origin xyz="0 -0.1 0.09" rpy="0 1.57 0"/>
         <geometry>
           <cylinder length="${wheel_width}" radius="${wheel_radius}"/>
@@ -78,9 +74,9 @@
         <origin xyz="0 0 0" rpy="0 0 0"/>
         <geometry>
-            <mesh filename="file:///$(find rocket)/meshes/M_rodatrativa.dae" scale="1 1 1"/>
+            <mesh filename="file:////home/renata_a/workspace/src/rocket/meshes/M_rodatrativa.dae" scale="1 1 1"/>
         </geometry>
       </visual>
       <collision name="right_wheel_collision">
-        <origin xyz="0 0 0" rpy="0 0 1.57"/>
+        <origin xyz="0 -0.1 0.09" rpy="0 1.57 0"/>
         <geometry>
           <cylinder length="${wheel_width}" radius="${wheel_radius}"/>
@@ -107,11 +103,11 @@
         <origin xyz="0 0 0.0118" rpy="0 0 0"/>
         <geometry>
-            <mesh filename="file:///$(find rocket)/meshes/ELV_conjuntocompleto.dae" scale="1 1 1"/>
+            <mesh filename="file:////home/renata_a/workspace/src/rocket/meshes/ELV_conjuntocompleto.dae" scale="1 1 1"/>
         </geometry>
       </visual>
       <collision name="tray_collision">
-        <origin xyz="0 0 0" rpy="0 0 0"/>
+        <origin xyz="0 -0.015047 0.1" rpy="0 0 0"/>
         <geometry>
-          <mesh filename="file:///$(find rocket)/meshes/ELV_conjuntocompleto.dae" scale="1 1 1"/>
+          <cylinder length="${tray_width}" radius="${tray_radius}"/>
         </geometry>
       </collision>
@@ -127,5 +123,5 @@
             <parent link="chassis" />
             <child link="tray" />
-            <origin rpy="0 0 0" xyz="0 0 0" />
+            <origin rpy="0 0 0" xyz="0 0.015047 0" />
     </joint>
 </robot>

Commit message: Ajeitei o path

File: urdf/robozinho.urdf.xacro (robot description, xacro)
@@ -24,5 +24,5 @@
         <origin xyz="0  0  0" rpy="0 0 0"/>
         <geometry>
-          <mesh filename="file:////home/renata_a/workspace/src/rocket/meshes/EST_estrutura_m3.dae" />
+          <mesh filename="file:///$(find rocket)/meshes/EST_estrutura_m3.dae" />
         </geometry>
       </visual>
@@ -46,5 +46,5 @@
         <origin xyz="0 0 0" rpy="0 0 0"/>
         <geometry>
-            <mesh filename="file:////home/renata_a/workspace/src/rocket/meshes/M_rodatrativa.dae" scale="1 1 1"/>
+            <mesh filename="file:///$(find rocket)/meshes/M_rodatrativa.dae" scale="1 1 1"/>
         </geometry>
       </visual>
@@ -74,5 +74,5 @@
         <origin xyz="0 0 0" rpy="0 0 0"/>
         <geometry>
-            <mesh filename="file:////home/renata_a/workspace/src/rocket/meshes/M_rodatrativa.dae" scale="1 1 1"/>
+            <mesh filename="file:///$(find rocket)/meshes/M_rodatrativa.dae" scale="1 1 1"/>
         </geometry>
       </visual>
@@ -103,5 +103,5 @@
         <origin xyz="0 0 0.0118" rpy="0 0 0"/>
         <geometry>
-            <mesh filename="file:////home/renata_a/workspace/src/rocket/meshes/ELV_conjuntocompleto.dae" scale="1 1 1"/>
+            <mesh filename="file:///$(find rocket)/meshes/ELV_conjuntocompleto.dae" scale="1 1 1"/>
         </geometry>
       </visual>

Commit message: Inercia

File: urdf/robozinho.urdf.xacro (robot description, xacro)
@@ -34,5 +34,5 @@
       </collision>
       <inertial>
-          <origin xyz="0  0  0.0118" rpy="0  0  3.14"/>
+          <origin xyz="0  0  -0.0118" rpy="0  0  0"/>
           <mass value="2.4"/>
           <inertia ixx="0.019995" ixy="0.0" ixz="0.0"
@@ -57,5 +57,5 @@
       <inertial>
         <mass value="1" />
-        <origin rpy="0 0 0" xyz="0 0 0" />
+        <origin rpy="0 1.57 0" xyz="0 -0.1 0.09" />
         <inertia ixx="0.001" ixy="0.0" ixz="0.0"
                 iyy="0.001" iyz="0.0"
@@ -85,5 +85,5 @@
       <inertial>
         <mass value="1" />
-        <origin rpy="0 0 0" xyz="0 0 0" />
+        <origin rpy="0 1.57 0" xyz="0 -0.1 0.09" />
         <inertia ixx="0.001" ixy="0.0" ixz="0.0"
                 iyy="0.001" iyz="0.0"
@@ -114,5 +114,5 @@
       <inertial>
         <mass value="0.5" />
-        <origin rpy="0 0 0" xyz="0 0 0" />
+        <origin rpy="0 0 0" xyz="0 -0.015047 0.1" />
         <inertia ixx="0.0" ixy="0.0" ixz="0.0"
                 iyy="0.0" iyz="0.0"

Commit message: troquei a roda pra continua mas o rviz ainda nao funciona

File: urdf/robozinho.urdf.xacro (robot description, xacro)
@@ -63,10 +63,9 @@
       </inertial>
     </link>
-    <joint name="joint_left_wheel" type="revolute">
+    <joint name="joint_left_wheel" type="continuous">
             <parent link="chassis" />
             <child link="left_wheel" />
             <origin rpy="0 0 1.57" xyz="-0.098795 -0.296755 -0.09915" />
             <axis rpy="0 0 0" xyz="0 1 0"/>
-            <limit effort="10000" velocity="1000"/>
     </joint>
     <link name="right_wheel">
@@ -91,10 +90,9 @@
       </inertial>
     </link>
-    <joint name="joint_right_wheel" type="revolute">
+    <joint name="joint_right_wheel" type="continuous">
             <parent link="chassis" />
             <child link="right_wheel" />
             <origin rpy="0 0 1.57" xyz="-0.098795 0.296395 -0.09915" />
             <axis rpy="0 0 0" xyz="0 1 0"/>
-            <limit effort="10000" velocity="1000"/>
     </joint>
   <!-- *********************** TRAY ******************************  -->

Commit message: arrumei um monte de coisa e agora ele anda

File: urdf/robozinho.urdf.xacro (robot description, xacro)
@@ -3,7 +3,7 @@
   <!-- ****************** ROBOT CONSTANTS *******************************  -->
   <!-- Define the size of the robot's main chassis in meters -->
-  <xacro:property name="base_width" value="0.557"/>
-  <xacro:property name="base_length" value="0.617"/>
-  <xacro:property name="base_height" value="0.1305"/>
+  <xacro:property name="base_width" value="0.47"/>
+  <xacro:property name="base_length" value="0.77"/>
+  <xacro:property name="base_height" value="0.15"/>
   <!-- Define the shape of the robot's two wheels in meters -->
   <xacro:property name="wheel_radius" value="0.07"/>
@@ -28,5 +28,5 @@
       </visual>
       <collision>
-          <origin rpy="0  0  0" xyz="0  0  -0.0118" />
+          <origin rpy="0  0  0" xyz="0  0  0.01" />
           <geometry>
               <box size="${base_length} ${base_width} ${base_height}"/>
@@ -50,5 +50,5 @@
       </visual>
       <collision name="left_wheel_collision">
-        <origin xyz="0 -0.1 0.09" rpy="0 1.57 0"/>
+        <origin xyz="0 0 0" rpy="0 1.57 0"/>
         <geometry>
           <cylinder length="${wheel_width}" radius="${wheel_radius}"/>
@@ -57,5 +57,5 @@
       <inertial>
         <mass value="1" />
-        <origin rpy="0 1.57 0" xyz="0 -0.1 0.09" />
+        <origin rpy="0 1.57 0" xyz="0 0 0" />
         <inertia ixx="0.001" ixy="0.0" ixz="0.0"
                 iyy="0.001" iyz="0.0"
@@ -66,6 +66,6 @@
             <parent link="chassis" />
             <child link="left_wheel" />
-            <origin rpy="0 0 1.57" xyz="-0.098795 -0.296755 -0.09915" />
-            <axis rpy="0 0 0" xyz="0 1 0"/>
+            <origin rpy="0 0 1.57" xyz=" 0 -0.296755 0" />
+            <axis rpy="0 0 0" xyz="1 0 0"/>
     </joint>
     <link name="right_wheel">
@@ -77,5 +77,5 @@
       </visual>
       <collision name="right_wheel_collision">
-        <origin xyz="0 -0.1 0.09" rpy="0 1.57 0"/>
+        <origin xyz="0 0 0" rpy="0 1.57 0"/>
         <geometry>
           <cylinder length="${wheel_width}" radius="${wheel_radius}"/>
@@ -84,5 +84,5 @@
       <inertial>
         <mass value="1" />
-        <origin rpy="0 1.57 0" xyz="0 -0.1 0.09" />
+        <origin rpy="0 1.57 0" xyz="0 0 0" />
         <inertia ixx="0.001" ixy="0.0" ixz="0.0"
                 iyy="0.001" iyz="0.0"
@@ -93,6 +93,6 @@
             <parent link="chassis" />
             <child link="right_wheel" />
-            <origin rpy="0 0 1.57" xyz="-0.098795 0.296395 -0.09915" />
-            <axis rpy="0 0 0" xyz="0 1 0"/>
+            <origin rpy="0 0 1.57" xyz="0 0.296395 0" />
+            <axis rpy="0 0 0" xyz="1 0 0"/>
     </joint>
   <!-- *********************** TRAY ******************************  -->
