Commit message: tentando colocar controle e falhando miseravelmente

File: urdf/rocket.urdf.xacro (robot description, xacro)
@@ -1,4 +1,8 @@
 <?xml version="1.0" ?>
-<robot name="robozinho" xmlns:xacro="http://ros.org/wiki/xacro">
+<robot name="rocket" xmlns:xacro="http://ros.org/wiki/xacro">
+  <!--=========================== CONTROL ===========================-->
+  <xacro:include filename="$(find rocket)/urdf/rocket_control.xacro" />
+  <!--=========================== PLUGINS ===========================-->
+  <!-- <xacro:include filename="$(find rocket)/urdf/rocket.gazebo.xacro" /> -->
   <!-- ****************** ROBOT CONSTANTS *******************************  -->
   <!-- Define the size of the robot's main chassis in meters -->
@@ -122,9 +126,4 @@
             <child link="tray" />
             <origin rpy="0 0 0" xyz="0 0.015047 0" />
-    </joint>
-  <gazebo>
-    <plugin name="gazebo_ros_control" filename="libgazebo_ros_control.so">
-      <robotNamespace>/</robotNamespace>
-    </plugin>
-  </gazebo>
+  </joint>
 </robot>

Commit message: Precisa ajeitar roda boba e referencias

File: urdf/rocket.urdf.xacro (robot description, xacro)
@@ -9,5 +9,5 @@
   <xacro:property name="base_width" value="0.47"/>
   <xacro:property name="base_length" value="0.77"/>
-  <xacro:property name="base_height" value="0.15"/>
+  <xacro:property name="base_height" value="0.13"/>
   <!-- Define the shape of the robot's two wheels in meters -->
   <xacro:property name="wheel_radius" value="0.07"/>
@@ -19,4 +19,12 @@
   <link name="base_link">
     </link>
+    <gazebo reference="chassis">
+      <selfCollide>true</selfCollide>
+      <mu1 value="0.3" />
+      <mu2 value="0.3" />
+      <kp value="1000000.0" />
+      <kd value="100" />
+      <fdir1 value="0 0 0" />
+    </gazebo>
     <joint name="base_joint" type="fixed">
       <parent link="base_link"/>
@@ -38,12 +46,21 @@
       </collision>
       <inertial>
-          <origin xyz="0  0  -0.0118" rpy="0  0  0"/>
+          <origin xyz="0  0  0" rpy="0  1.57  0"/>
           <mass value="2.4"/>
-          <inertia ixx="0.019995" ixy="0.0" ixz="0.0"
-                iyy="0.019995" iyz="0.0"
-                izz="0.03675" />
+          <inertia ixx="0.12196" ixy="0.0" ixz="0.0"
+                iyy="0.16276" iyz="0.0"
+                izz="0.14756" />
       </inertial>
     </link>
   <!-- *********************** DRIVE WHEELS ******************************  -->
+    <gazebo reference="left_wheel">
+      <selfCollide>false</selfCollide>
+      <mu1>1.0</mu1>
+      <mu2>1.0</mu2>
+      <kp>1000000.0</kp>
+      <kd>100.0</kd>
+      <maxVel>1.0</maxVel>
+      <fdir1 value="0 0 0" />
+    </gazebo>
     <link name="left_wheel">
       <visual name="left_wheel_visual">
@@ -73,4 +90,13 @@
             <axis rpy="0 0 0" xyz="1 0 0"/>
     </joint>
+    <gazebo reference="right_wheel">
+      <selfCollide>false</selfCollide>
+      <mu1>1.0</mu1>
+      <mu2>1.0</mu2>
+      <kp>1000000.0</kp>
+      <kd>100.0</kd>
+      <maxVel>1.0</maxVel>
+      <fdir1 value="0 0 0" />
+    </gazebo>
     <link name="right_wheel">
       <visual name="right_wheel_visual">
@@ -116,5 +142,5 @@
       <inertial>
         <mass value="0.5" />
-        <origin rpy="0 0 0" xyz="0 -0.015047 0.1" />
+        <origin rpy="0 0 0" xyz="0 0 0" />
         <inertia ixx="0.0" ixy="0.0" ixz="0.0"
                 iyy="0.0" iyz="0.0"
@@ -127,3 +153,152 @@
             <origin rpy="0 0 0" xyz="0 0.015047 0" />
   </joint>
+  <!-- *********************** CASTER WHEELS ******************************  -->
+  <gazebo reference="back_left_caster_wheel">
+      <selfCollide>true</selfCollide>
+      <mu1 value="0.09" />
+      <mu2 value="0.09" />
+      <kp value="10000000.0" />
+      <kd value="10000" />
+      <fdir1 value="0 0 0" />
+  </gazebo>
+  <link name="back_left_caster_wheel">
+    <visual name="back_left_caster_wheel_visual">
+      <origin xyz="0 0 0" rpy="0 0 0"/>
+      <geometry>
+        <sphere radius="0.01"/>
+      </geometry>
+      <material name="Black">
+          <color rgba="${0/255} ${0/255} ${0/255} 1.0"/>
+     </material>
+    </visual>
+    <collision name="back_left_caster_wheel_collision">
+      <origin xyz="0 0 0" rpy="0 0 0"/>
+      <geometry>
+        <sphere radius="0.01"/>
+      </geometry>
+    </collision>
+    <inertial>
+        <mass value="0.1" />
+        <origin rpy="0 0 0" xyz="0 0 0" />
+        <inertia ixx="0" ixy="0.0" ixz="0.0"
+                iyy="0" iyz="0.0"
+                izz="0" />
+      </inertial>
+  </link>
+  <joint name="joint_back_left_caster_wheel" type="fixed">
+    <parent link="chassis"/>
+    <child link="back_left_caster_wheel"/>
+    <origin rpy="0 0 0" xyz="0.32 0.07 -0.06"/>
+  </joint>
+  <gazebo reference="back_right_caster_wheel">
+      <selfCollide>true</selfCollide>
+      <mu1 value="0.09" />
+      <mu2 value="0.09" />
+      <kp value="10000000.0" />
+      <kd value="10000" />
+      <fdir1 value="0 0 0" />
+  </gazebo>
+  <link name="back_right_caster_wheel">
+    <visual name="back_right_caster_wheel_visual">
+      <origin xyz="0 0 0" rpy="0 0 0"/>
+      <geometry>
+        <sphere radius="0.01"/>
+      </geometry>
+      <material name="Black">
+          <color rgba="${0/255} ${0/255} ${0/255} 1.0"/>
+     </material>
+    </visual>
+    <collision name="back_right_caster_wheel_collision">
+      <origin xyz="0 0 0" rpy="0 0 0"/>
+      <geometry>
+        <sphere radius="0.01"/>
+      </geometry>
+    </collision>
+    <inertial>
+        <mass value="0.1" />
+        <origin rpy="0 0 0" xyz="0 0 0" />
+        <inertia ixx="0" ixy="0.0" ixz="0.0"
+                iyy="0" iyz="0.0"
+                izz="0" />
+      </inertial>
+  </link>
+  <joint name="joint_back_right_caster_wheel" type="fixed">
+    <parent link="chassis"/>
+    <child link="back_right_caster_wheel"/>
+    <origin rpy="0 0 0" xyz="0.32 -0.07 -0.06"/>
+  </joint>
+  <gazebo reference="front_left_caster_wheel">
+      <selfCollide>true</selfCollide>
+      <mu1 value="0.09" />
+      <mu2 value="0.09" />
+      <kp value="10000000.0" />
+      <kd value="10000" />
+      <fdir1 value="0 0 0" />
+  </gazebo>
+  <link name="front_left_caster_wheel">
+    <visual name="front_left_caster_wheel_visual">
+      <origin xyz="0 0 0" rpy="0 0 0"/>
+      <geometry>
+        <sphere radius="0.01"/>
+      </geometry>
+      <material name="Black">
+          <color rgba="${0/255} ${0/255} ${0/255} 1.0"/>
+     </material>
+    </visual>
+    <collision name="front_left_caster_wheel_collision">
+      <origin xyz="0 0 0" rpy="0 0 0"/>
+      <geometry>
+        <sphere radius="0.01"/>
+      </geometry>
+    </collision>
+    <inertial>
+        <mass value="0.1" />
+        <origin rpy="0 0 0" xyz="0 0 0" />
+        <inertia ixx="0" ixy="0.0" ixz="0.0"
+                iyy="0" iyz="0.0"
+                izz="0" />
+      </inertial>
+  </link>
+  <joint name="joint_front_left_caster_wheel" type="fixed">
+    <parent link="chassis"/>
+    <child link="front_left_caster_wheel"/>
+    <origin rpy="0 0 0" xyz="-0.32 0.07 -0.06"/>
+  </joint>
+  <gazebo reference="front_right_caster_wheel">
+      <selfCollide>true</selfCollide>
+      <mu1 value="0.09" />
+      <mu2 value="0.09" />
+      <kp value="10000000.0" />
+      <kd value="10000" />
+      <fdir1 value="0 0 0" />
+  </gazebo>
+  <link name="front_right_caster_wheel">
+    <visual name="front_right_caster_wheel_visual">
+      <origin xyz="0 0 0" rpy="0 0 0"/>
+      <geometry>
+        <sphere radius="0.01"/>
+      </geometry>
+      <material name="Black">
+          <color rgba="${0/255} ${0/255} ${0/255} 1.0"/>
+     </material>
+    </visual>
+    <collision name="front_right_caster_wheel_collision">
+      <origin xyz="0 0 0" rpy="0 0 0"/>
+      <geometry>
+        <sphere radius="0.01"/>
+      </geometry>
+    </collision>
+    <inertial>
+        <mass value="0.1" />
+        <origin rpy="0 0 0" xyz="0 0 0" />
+        <inertia ixx="0" ixy="0.0" ixz="0.0"
+                iyy="0" iyz="0.0"
+                izz="0" />
+      </inertial>
+  </link>
+  <joint name="joint_front_right_caster_wheel" type="fixed">
+    <parent link="chassis"/>
+    <child link="front_right_caster_wheel"/>
+    <origin rpy="0 0 0" xyz="-0.32 -0.07 -0.06"/>
+  </joint>
 </robot>

Commit message: consegui arrumar o controle e fazer o teleop funcionar, so falta arrumar as rodas bobas e criar um launch pra o teleop

File: urdf/rocket.urdf.xacro (robot description, xacro)
@@ -2,5 +2,5 @@
 <robot name="rocket" xmlns:xacro="http://ros.org/wiki/xacro">
   <!--=========================== CONTROL ===========================-->
-  <xacro:include filename="$(find rocket)/urdf/rocket_control.xacro" />
+  <xacro:include filename="rocket_control.xacro" />
   <!--=========================== PLUGINS ===========================-->
   <!-- <xacro:include filename="$(find rocket)/urdf/rocket.gazebo.xacro" /> -->

File: urdf/rocket_control.xacro (robot description, xacro)
@@ -5,5 +5,5 @@
             <plugin>gazebo_ros2_control/GazeboSystem</plugin>
         </hardware>
-        <joint name="left_wheel_joint">
+        <joint name="joint_left_wheel">
             <command_interface name="velocity">
                 <param name="min">-10</param>
@@ -13,5 +13,5 @@
             <state_interface name="position"/>
         </joint>
-                <joint name="right_wheel_joint">
+        <joint name="joint_right_wheel">
             <command_interface name="velocity">
                 <param name="min">-10</param>

Commit message: Rodas ajeitadas

File: urdf/rocket.urdf.xacro (robot description, xacro)
@@ -11,14 +11,20 @@
   <xacro:property name="base_height" value="0.13"/>
   <!-- Define the shape of the robot's two wheels in meters -->
-  <xacro:property name="wheel_radius" value="0.07"/>
+  <xacro:property name="wheel_radius" value="0.08"/>
   <xacro:property name="wheel_width" value="0.03"/>
   <!-- Define the shape of the robot's tray in meters -->
   <xacro:property name="tray_radius" value="0.2"/>
   <xacro:property name="tray_width" value="0.041"/>
+  <!-- Define the shape of the robot's four caster wheels in meters -->
+  <xacro:property name="caster_wheel_radius" value="0.01"/>
+  <!-- Colors -->
+  <material name="black">
+      <color rgba="0.0 0.0 0.0 1.0"/>
+  </material>
   <!-- ********************** ROBOT BASE *********************************  -->
   <link name="base_link">
     </link>
     <gazebo reference="chassis">
-      <selfCollide>true</selfCollide>
+      <!-- <selfCollide>true</selfCollide> -->
       <mu1 value="0.3" />
       <mu2 value="0.3" />
@@ -49,17 +55,17 @@
           <mass value="2.4"/>
           <inertia ixx="0.12196" ixy="0.0" ixz="0.0"
-                iyy="0.16276" iyz="0.0"
-                izz="0.14756" />
+                iyy="0.04756" iyz="0.0"
+                izz="0.16276" />
       </inertial>
     </link>
   <!-- *********************** DRIVE WHEELS ******************************  -->
     <gazebo reference="left_wheel">
-      <selfCollide>false</selfCollide>
+      <!-- <selfCollide>false</selfCollide> -->
       <mu1>1.0</mu1>
       <mu2>1.0</mu2>
       <kp>1000000.0</kp>
       <kd>100.0</kd>
-      <maxVel>1.0</maxVel>
-      <fdir1 value="0 0 0" />
+      <!-- <maxVel>1.0</maxVel> -->
+      <!-- <fdir1 value="0 0 0" /> -->
     </gazebo>
     <link name="left_wheel">
@@ -79,7 +85,7 @@
         <mass value="1" />
         <origin rpy="0 1.57 0" xyz="0 0 0" />
-        <inertia ixx="0.001" ixy="0.0" ixz="0.0"
-                iyy="0.001" iyz="0.0"
-                izz="0.001" />
+        <inertia ixx="0.0013" ixy="0.0" ixz="0.0"
+                iyy="0.0013" iyz="0.0"
+                izz="0.00245" />
       </inertial>
     </link>
@@ -91,11 +97,11 @@
     </joint>
     <gazebo reference="right_wheel">
-      <selfCollide>false</selfCollide>
+      <!-- <selfCollide>false</selfCollide> -->
       <mu1>1.0</mu1>
       <mu2>1.0</mu2>
       <kp>1000000.0</kp>
       <kd>100.0</kd>
-      <maxVel>1.0</maxVel>
-      <fdir1 value="0 0 0" />
+      <!-- <maxVel>1.0</maxVel> -->
+      <!-- <fdir1 value="0 0 0" /> -->
     </gazebo>
     <link name="right_wheel">
@@ -115,7 +121,7 @@
         <mass value="1" />
         <origin rpy="0 1.57 0" xyz="0 0 0" />
-        <inertia ixx="0.001" ixy="0.0" ixz="0.0"
-                iyy="0.001" iyz="0.0"
-                izz="0.001" />
+        <inertia ixx="0.0013" ixy="0.0" ixz="0.0"
+                iyy="0.0013" iyz="0.0"
+                izz="0.00245" />
       </inertial>
     </link>
@@ -160,5 +166,5 @@
       <kp value="10000000.0" />
       <kd value="10000" />
-      <fdir1 value="0 0 0" />
+      <!-- <fdir1 value="0 0 0" /> -->
   </gazebo>
   <link name="back_left_caster_wheel">
@@ -166,9 +172,7 @@
       <origin xyz="0 0 0" rpy="0 0 0"/>
       <geometry>
-        <sphere radius="0.01"/>
-      </geometry>
-      <material name="Black">
-          <color rgba="${0/255} ${0/255} ${0/255} 1.0"/>
-     </material>
+        <sphere radius="${caster_wheel_radius}"/>
+      </geometry>
+      <material name="black"/>
     </visual>
     <collision name="back_left_caster_wheel_collision">
@@ -179,15 +183,15 @@
     </collision>
     <inertial>
-        <mass value="0.1" />
-        <origin rpy="0 0 0" xyz="0 0 0" />
-        <inertia ixx="0" ixy="0.0" ixz="0.0"
-                iyy="0" iyz="0.0"
-                izz="0" />
-      </inertial>
+      <origin xyz="0 0 0" />
+      <mass value="0.005" />
+      <inertia ixx="0.001" ixy="0.0" ixz="0.0"
+               iyy="0.001" iyz="0.0"
+               izz="0.001" />
+    </inertial>
   </link>
   <joint name="joint_back_left_caster_wheel" type="fixed">
     <parent link="chassis"/>
     <child link="back_left_caster_wheel"/>
-    <origin rpy="0 0 0" xyz="0.32 0.07 -0.06"/>
+    <origin rpy="-1.57 0 0" xyz="0.32 0.07 -0.06"/>
   </joint>
   <gazebo reference="back_right_caster_wheel">
@@ -197,5 +201,5 @@
       <kp value="10000000.0" />
       <kd value="10000" />
-      <fdir1 value="0 0 0" />
+      <!-- <fdir1 value="0 0 0" /> -->
   </gazebo>
   <link name="back_right_caster_wheel">
@@ -203,9 +207,7 @@
       <origin xyz="0 0 0" rpy="0 0 0"/>
       <geometry>
-        <sphere radius="0.01"/>
-      </geometry>
-      <material name="Black">
-          <color rgba="${0/255} ${0/255} ${0/255} 1.0"/>
-     </material>
+        <sphere radius="${caster_wheel_radius}"/>
+      </geometry>
+      <material name="black"/>
     </visual>
     <collision name="back_right_caster_wheel_collision">
@@ -216,15 +218,15 @@
     </collision>
     <inertial>
-        <mass value="0.1" />
-        <origin rpy="0 0 0" xyz="0 0 0" />
-        <inertia ixx="0" ixy="0.0" ixz="0.0"
-                iyy="0" iyz="0.0"
-                izz="0" />
-      </inertial>
+      <origin xyz="0 0 0" />
+      <mass value="0.005" />
+      <inertia ixx="0.001" ixy="0.0" ixz="0.0"
+               iyy="0.001" iyz="0.0"
+               izz="0.001" />
+    </inertial>
   </link>
   <joint name="joint_back_right_caster_wheel" type="fixed">
     <parent link="chassis"/>
     <child link="back_right_caster_wheel"/>
-    <origin rpy="0 0 0" xyz="0.32 -0.07 -0.06"/>
+    <origin rpy="-1.57 0 0" xyz="0.32 -0.07 -0.06"/>
   </joint>
   <gazebo reference="front_left_caster_wheel">
@@ -234,5 +236,5 @@
       <kp value="10000000.0" />
       <kd value="10000" />
-      <fdir1 value="0 0 0" />
+      <!-- <fdir1 value="0 0 0" /> -->
   </gazebo>
   <link name="front_left_caster_wheel">
@@ -240,9 +242,7 @@
       <origin xyz="0 0 0" rpy="0 0 0"/>
       <geometry>
-        <sphere radius="0.01"/>
-      </geometry>
-      <material name="Black">
-          <color rgba="${0/255} ${0/255} ${0/255} 1.0"/>
-     </material>
+        <sphere radius="${caster_wheel_radius}"/>
+      </geometry>
+      <material name="black"/>
     </visual>
     <collision name="front_left_caster_wheel_collision">
@@ -253,15 +253,15 @@
     </collision>
     <inertial>
-        <mass value="0.1" />
-        <origin rpy="0 0 0" xyz="0 0 0" />
-        <inertia ixx="0" ixy="0.0" ixz="0.0"
-                iyy="0" iyz="0.0"
-                izz="0" />
-      </inertial>
+      <origin xyz="0 0 0" />
+      <mass value="0.005" />
+      <inertia ixx="0.001" ixy="0.0" ixz="0.0"
+               iyy="0.001" iyz="0.0"
+               izz="0.001" />
+        </inertial>
   </link>
   <joint name="joint_front_left_caster_wheel" type="fixed">
     <parent link="chassis"/>
     <child link="front_left_caster_wheel"/>
-    <origin rpy="0 0 0" xyz="-0.32 0.07 -0.06"/>
+    <origin rpy="-1.57 0 0" xyz="-0.32 0.07 -0.06"/>
   </joint>
   <gazebo reference="front_right_caster_wheel">
@@ -271,5 +271,5 @@
       <kp value="10000000.0" />
       <kd value="10000" />
-      <fdir1 value="0 0 0" />
+      <!-- <fdir1 value="0 0 0" /> -->
   </gazebo>
   <link name="front_right_caster_wheel">
@@ -277,9 +277,7 @@
       <origin xyz="0 0 0" rpy="0 0 0"/>
       <geometry>
-        <sphere radius="0.01"/>
-      </geometry>
-      <material name="Black">
-          <color rgba="${0/255} ${0/255} ${0/255} 1.0"/>
-     </material>
+        <sphere radius="${caster_wheel_radius}"/>
+      </geometry>
+      <material name="black"/>
     </visual>
     <collision name="front_right_caster_wheel_collision">
@@ -290,15 +288,15 @@
     </collision>
     <inertial>
-        <mass value="0.1" />
-        <origin rpy="0 0 0" xyz="0 0 0" />
-        <inertia ixx="0" ixy="0.0" ixz="0.0"
-                iyy="0" iyz="0.0"
-                izz="0" />
-      </inertial>
+      <origin xyz="0 0 0" />
+      <mass value="0.005" />
+      <inertia ixx="0.001" ixy="0.0" ixz="0.0"
+               iyy="0.001" iyz="0.0"
+               izz="0.001" />
+    </inertial>
   </link>
   <joint name="joint_front_right_caster_wheel" type="fixed">
     <parent link="chassis"/>
     <child link="front_right_caster_wheel"/>
-    <origin rpy="0 0 0" xyz="-0.32 -0.07 -0.06"/>
+    <origin rpy="-1.57 0 0" xyz="-0.32 -0.07 -0.06"/>
   </joint>
 </robot>

Commit message: eu sla oq mudei

File: urdf/rocket.urdf.xacro (robot description, xacro)
@@ -11,5 +11,5 @@
   <xacro:property name="base_height" value="0.13"/>
   <!-- Define the shape of the robot's two wheels in meters -->
-  <xacro:property name="wheel_radius" value="0.08"/>
+  <xacro:property name="wheel_radius" value="0.07"/>
   <xacro:property name="wheel_width" value="0.03"/>
   <!-- Define the shape of the robot's tray in meters -->
@@ -26,5 +26,4 @@
     </link>
     <gazebo reference="chassis">
-      <!-- <selfCollide>true</selfCollide> -->
       <mu1 value="0.3" />
       <mu2 value="0.3" />
@@ -36,5 +35,5 @@
       <parent link="base_link"/>
       <child link="chassis" />
-      <origin xyz="0.0 0.0 0.0118" rpy="0 0 3.14"/>
+      <origin xyz="0.0 0.0 0.0" rpy="0 0 3.14"/>
     </joint>
     <link name="chassis">
@@ -61,11 +60,8 @@
   <!-- *********************** DRIVE WHEELS ******************************  -->
     <gazebo reference="left_wheel">
-      <!-- <selfCollide>false</selfCollide> -->
       <mu1>1.0</mu1>
       <mu2>1.0</mu2>
       <kp>1000000.0</kp>
       <kd>100.0</kd>
-      <!-- <maxVel>1.0</maxVel> -->
-      <!-- <fdir1 value="0 0 0" /> -->
     </gazebo>
     <link name="left_wheel">
@@ -93,5 +89,5 @@
             <parent link="chassis" />
             <child link="left_wheel" />
-            <origin rpy="0 0 1.57" xyz=" 0 -0.296755 0" />
+            <origin rpy="0 0 1.57" xyz=" 0 -0.296755 -0.0118" />
             <axis rpy="0 0 0" xyz="1 0 0"/>
     </joint>
@@ -129,5 +125,5 @@
             <parent link="chassis" />
             <child link="right_wheel" />
-            <origin rpy="0 0 1.57" xyz="0 0.296395 0" />
+            <origin rpy="0 0 1.57" xyz="0 0.296395 -0.0118" />
             <axis rpy="0 0 0" xyz="1 0 0"/>
     </joint>
@@ -166,5 +162,4 @@
       <kp value="10000000.0" />
       <kd value="10000" />
-      <!-- <fdir1 value="0 0 0" /> -->
   </gazebo>
   <link name="back_left_caster_wheel">
