Commit message: a gente arrumou um monte do urdf

File: urdf/rocket.urdf.xacro (robot description, xacro)
@@ -6,11 +6,11 @@
   <!-- <xacro:include filename="$(find rocket)/urdf/rocket.gazebo.xacro" /> -->
   <!-- ****************** ROBOT CONSTANTS *******************************  -->
-  <!-- Define the size of the robot's main chassis in meters -->
+  <!-- Define the size of the robot's main base_link in meters -->
   <xacro:property name="base_width" value="0.47"/>
   <xacro:property name="base_length" value="0.77"/>
   <xacro:property name="base_height" value="0.13"/>
   <!-- Define the shape of the robot's two wheels in meters -->
-  <xacro:property name="wheel_radius" value="0.07"/>
-  <xacro:property name="wheel_width" value="0.03"/>
+  <xacro:property name="wheel_radius" value="0.0675"/>
+  <xacro:property name="wheel_width" value="0.04"/>
   <!-- Define the shape of the robot's tray in meters -->
   <xacro:property name="tray_radius" value="0.2"/>
@@ -23,7 +23,7 @@
   </material>
   <!-- ********************** ROBOT BASE *********************************  -->
-  <link name="base_link">
-    </link>
-    <gazebo reference="chassis">
+  <link name="base_footprint">
+    </link>
+    <gazebo reference="base_link">
       <mu1 value="0.3" />
       <mu2 value="0.3" />
@@ -34,8 +34,8 @@
     <joint name="base_joint" type="fixed">
       <parent link="base_link"/>
-      <child link="chassis" />
-      <origin xyz="0.0 0.0 0.0" rpy="0 0 3.14"/>
+      <child link="base_footprint" />
+      <origin xyz="0.0 0.0 -0.0793" rpy="0 0 3.14"/>
     </joint>
-    <link name="chassis">
+    <link name="base_link">
       <visual>
         <origin xyz="0  0  0" rpy="0 0 0"/>
@@ -87,5 +87,5 @@
     </link>
     <joint name="joint_left_wheel" type="continuous">
-            <parent link="chassis" />
+            <parent link="base_link" />
             <child link="left_wheel" />
             <origin rpy="0 0 1.57" xyz=" 0 -0.296755 -0.0118" />
@@ -123,5 +123,5 @@
     </link>
     <joint name="joint_right_wheel" type="continuous">
-            <parent link="chassis" />
+            <parent link="base_link" />
             <child link="right_wheel" />
             <origin rpy="0 0 1.57" xyz="0 0.296395 -0.0118" />
@@ -151,5 +151,5 @@
   </link>
   <joint name="joint_tray" type="fixed">
-            <parent link="chassis" />
+            <parent link="base_link" />
             <child link="tray" />
             <origin rpy="0 0 0" xyz="0 0.015047 0" />
@@ -186,5 +186,5 @@
   </link>
   <joint name="joint_back_left_caster_wheel" type="fixed">
-    <parent link="chassis"/>
+    <parent link="base_link"/>
     <child link="back_left_caster_wheel"/>
     <origin rpy="-1.57 0 0" xyz="0.32 0.07 -0.06"/>
@@ -221,5 +221,5 @@
   </link>
   <joint name="joint_back_right_caster_wheel" type="fixed">
-    <parent link="chassis"/>
+    <parent link="base_link"/>
     <child link="back_right_caster_wheel"/>
     <origin rpy="-1.57 0 0" xyz="0.32 -0.07 -0.06"/>
@@ -256,5 +256,5 @@
   </link>
   <joint name="joint_front_left_caster_wheel" type="fixed">
-    <parent link="chassis"/>
+    <parent link="base_link"/>
     <child link="front_left_caster_wheel"/>
     <origin rpy="-1.57 0 0" xyz="-0.32 0.07 -0.06"/>
@@ -291,5 +291,5 @@
   </link>
   <joint name="joint_front_right_caster_wheel" type="fixed">
-    <parent link="chassis"/>
+    <parent link="base_link"/>
     <child link="front_right_caster_wheel"/>
     <origin rpy="-1.57 0 0" xyz="-0.32 -0.07 -0.06"/>
