Commit message: magica

File: urdf/l1br.urdf.xacro (robot description, xacro)
@@ -1,8 +1,10 @@
 <?xml version="1.0" ?>
-<robot name="rocket" xmlns:xacro="http://ros.org/wiki/xacro">
+<robot name="l1br" xmlns:xacro="http://ros.org/wiki/xacro">
   <!--=========================== CONTROL ===========================-->
-  <xacro:include filename="rocket_control.xacro" />
+  <xacro:include filename="l1br_control.xacro" />
+  <xacro:include filename="sensors/imu_sensor.urdf.xacro" />
+  <xacro:include filename="sensors/laser_sensor.urdf.xacro" />
   <!--=========================== PLUGINS ===========================-->
-  <!-- <xacro:include filename="$(find rocket)/urdf/rocket.gazebo.xacro" /> -->
+  <!-- <xacro:include filename="$(find l1br)/urdf/l1br.gazebo.xacro" /> -->
   <!-- ****************** ROBOT CONSTANTS *******************************  -->
   <!-- Define the size of the robot's main base_link in meters -->
@@ -41,5 +43,5 @@
         <origin xyz="0  0  0" rpy="0 0 0"/>
         <geometry>
-          <mesh filename="file:///$(find rocket)/meshes/EST_estrutura_m3.dae" />
+          <mesh filename="file:///$(find l1br)/meshes/EST_estrutura_m3.dae" />
         </geometry>
       </visual>
@@ -51,5 +53,5 @@
       </collision>
       <inertial>
-          <origin xyz="0  0  0" rpy="0  1.57  0"/>
+          <origin xyz="0  0  0.0" rpy="0 0 1.57"/>
           <mass value="2.4"/>
           <inertia ixx="0.12196" ixy="0.0" ixz="0.0"
@@ -69,5 +71,5 @@
         <origin xyz="0 0 0" rpy="0 0 0"/>
         <geometry>
-            <mesh filename="file:///$(find rocket)/meshes/M_rodatrativa.dae" scale="1 1 1"/>
+            <mesh filename="file:///$(find l1br)/meshes/M_rodatrativa.dae" scale="1 1 1"/>
         </geometry>
       </visual>
@@ -79,9 +81,9 @@
       </collision>
       <inertial>
-        <mass value="1" />
         <origin rpy="0 1.57 0" xyz="0 0 0" />
-        <inertia ixx="0.0013" ixy="0.0" ixz="0.0"
-                iyy="0.0013" iyz="0.0"
-                izz="0.00245" />
+        <mass value="1"/>
+        <inertia ixx="${(2/5) * 1 * (wheel_radius * wheel_radius)}" ixy="0" ixz="0"
+                iyy="${(2/5) * 1 * (wheel_radius * wheel_radius)}" iyz="0"
+                izz="${(2/5) * 1 * (wheel_radius * wheel_radius)}" />
       </inertial>
     </link>
@@ -89,5 +91,5 @@
             <parent link="base_link" />
             <child link="left_wheel" />
-            <origin rpy="0 0 1.57" xyz=" 0 -0.296755 -0.0118" />
+            <origin rpy="0 0 1.57" xyz=" 0 0.296755 -0.0118" />
             <axis rpy="0 0 0" xyz="1 0 0"/>
     </joint>
@@ -105,5 +107,5 @@
         <origin xyz="0 0 0" rpy="0 0 0"/>
         <geometry>
-            <mesh filename="file:///$(find rocket)/meshes/M_rodatrativa.dae" scale="1 1 1"/>
+            <mesh filename="file:///$(find l1br)/meshes/M_rodatrativa.dae" scale="1 1 1"/>
         </geometry>
       </visual>
@@ -115,9 +117,9 @@
       </collision>
       <inertial>
-        <mass value="1" />
         <origin rpy="0 1.57 0" xyz="0 0 0" />
-        <inertia ixx="0.0013" ixy="0.0" ixz="0.0"
-                iyy="0.0013" iyz="0.0"
-                izz="0.00245" />
+        <mass value="1"/>
+        <inertia ixx="${(2/5) * 1 * (wheel_radius * wheel_radius)}" ixy="0" ixz="0"
+                iyy="${(2/5) * 1 * (wheel_radius * wheel_radius)}" iyz="0"
+                izz="${(2/5) * 1 * (wheel_radius * wheel_radius)}" />
       </inertial>
     </link>
@@ -125,5 +127,5 @@
             <parent link="base_link" />
             <child link="right_wheel" />
-            <origin rpy="0 0 1.57" xyz="0 0.296395 -0.0118" />
+            <origin rpy="0 0 1.57" xyz="0 -0.296395 -0.0118" />
             <axis rpy="0 0 0" xyz="1 0 0"/>
     </joint>
@@ -133,5 +135,5 @@
         <origin xyz="0 0 0.0118" rpy="0 0 0"/>
         <geometry>
-            <mesh filename="file:///$(find rocket)/meshes/ELV_conjuntocompleto.dae" scale="1 1 1"/>
+            <mesh filename="file:///$(find l1br)/meshes/ELV_conjuntocompleto.dae" scale="1 1 1"/>
         </geometry>
       </visual>
@@ -157,5 +159,5 @@
   <!-- *********************** CASTER WHEELS ******************************  -->
   <gazebo reference="back_left_caster_wheel">
-      <selfCollide>true</selfCollide>
+      <selfCollide>false</selfCollide>
       <mu1 value="0.09" />
       <mu2 value="0.09" />
@@ -178,18 +180,19 @@
     </collision>
     <inertial>
-      <origin xyz="0 0 0" />
-      <mass value="0.005" />
-      <inertia ixx="0.001" ixy="0.0" ixz="0.0"
-               iyy="0.001" iyz="0.0"
-               izz="0.001" />
+      <origin xyz="0 0 0" rpy="0 0 0"/>
+      <mass value="0.005"/>
+      <inertia ixx="${(2/5) * 0.005 * (caster_wheel_radius * caster_wheel_radius)}" ixy="0" ixz="0"
+              iyy="${(2/5) * 0.005 * (caster_wheel_radius * caster_wheel_radius)}" iyz="0"
+              izz="${(2/5) * 0.005 * (caster_wheel_radius * caster_wheel_radius)}" />
     </inertial>
   </link>
-  <joint name="joint_back_left_caster_wheel" type="fixed">
+  <joint name="joint_back_left_caster_wheel" type="continuous">
     <parent link="base_link"/>
     <child link="back_left_caster_wheel"/>
-    <origin rpy="-1.57 0 0" xyz="0.32 0.07 -0.06"/>
+    <origin rpy="-1.57 0 0" xyz="0.32 0.07 -0.0693"/>
+    <axis rpy="0 0 0" xyz="1 0 0"/>
   </joint>
   <gazebo reference="back_right_caster_wheel">
-      <selfCollide>true</selfCollide>
+      <selfCollide>false</selfCollide>
       <mu1 value="0.09" />
       <mu2 value="0.09" />
@@ -213,18 +216,19 @@
     </collision>
     <inertial>
-      <origin xyz="0 0 0" />
-      <mass value="0.005" />
-      <inertia ixx="0.001" ixy="0.0" ixz="0.0"
-               iyy="0.001" iyz="0.0"
-               izz="0.001" />
+      <origin xyz="0 0 0" rpy="0 0 0"/>
+      <mass value="0.005"/>
+      <inertia ixx="${(2/5) * 0.005 * (caster_wheel_radius * caster_wheel_radius)}" ixy="0" ixz="0"
+              iyy="${(2/5) * 0.005 * (caster_wheel_radius * caster_wheel_radius)}" iyz="0"
+              izz="${(2/5) * 0.005 * (caster_wheel_radius * caster_wheel_radius)}" />
     </inertial>
   </link>
-  <joint name="joint_back_right_caster_wheel" type="fixed">
+  <joint name="joint_back_right_caster_wheel" type="continuous">
     <parent link="base_link"/>
     <child link="back_right_caster_wheel"/>
-    <origin rpy="-1.57 0 0" xyz="0.32 -0.07 -0.06"/>
+    <origin rpy="-1.57 0 0" xyz="0.32 -0.07 -0.0693"/>
+    <axis rpy="0 0 0" xyz="1 0 0"/>
   </joint>
   <gazebo reference="front_left_caster_wheel">
-      <selfCollide>true</selfCollide>
+      <selfCollide>false</selfCollide>
       <mu1 value="0.09" />
       <mu2 value="0.09" />
@@ -248,18 +252,19 @@
     </collision>
     <inertial>
-      <origin xyz="0 0 0" />
-      <mass value="0.005" />
-      <inertia ixx="0.001" ixy="0.0" ixz="0.0"
-               iyy="0.001" iyz="0.0"
-               izz="0.001" />
-        </inertial>
-  </link>
-  <joint name="joint_front_left_caster_wheel" type="fixed">
+      <origin xyz="0 0 0" rpy="0 0 0"/>
+      <mass value="0.005"/>
+      <inertia ixx="${(2/5) * 0.005 * (caster_wheel_radius * caster_wheel_radius)}" ixy="0" ixz="0"
+              iyy="${(2/5) * 0.005 * (caster_wheel_radius * caster_wheel_radius)}" iyz="0"
+              izz="${(2/5) * 0.005 * (caster_wheel_radius * caster_wheel_radius)}" />
+    </inertial>
+  </link>
+  <joint name="joint_front_left_caster_wheel" type="continuous">
     <parent link="base_link"/>
     <child link="front_left_caster_wheel"/>
-    <origin rpy="-1.57 0 0" xyz="-0.32 0.07 -0.06"/>
+    <origin rpy="-1.57 0 0" xyz="-0.32 0.07 -0.0693"/>
+    <axis rpy="0 0 0" xyz="1 0 0"/>
   </joint>
   <gazebo reference="front_right_caster_wheel">
-      <selfCollide>true</selfCollide>
+      <selfCollide>false</selfCollide>
       <mu1 value="0.09" />
       <mu2 value="0.09" />
@@ -283,15 +288,29 @@
     </collision>
     <inertial>
-      <origin xyz="0 0 0" />
-      <mass value="0.005" />
-      <inertia ixx="0.001" ixy="0.0" ixz="0.0"
-               iyy="0.001" iyz="0.0"
-               izz="0.001" />
+      <origin xyz="0 0 0" rpy="0 0 0"/>
+      <mass value="0.005"/>
+      <inertia ixx="${(2/5) * 0.005 * (caster_wheel_radius * caster_wheel_radius)}" ixy="0" ixz="0"
+              iyy="${(2/5) * 0.005 * (caster_wheel_radius * caster_wheel_radius)}" iyz="0"
+              izz="${(2/5) * 0.005 * (caster_wheel_radius * caster_wheel_radius)}" />
     </inertial>
   </link>
-  <joint name="joint_front_right_caster_wheel" type="fixed">
+  <joint name="joint_front_right_caster_wheel" type="continuous">
     <parent link="base_link"/>
     <child link="front_right_caster_wheel"/>
-    <origin rpy="-1.57 0 0" xyz="-0.32 -0.07 -0.06"/>
-  </joint>
+    <origin rpy="-1.57 0 0" xyz="-0.32 -0.07 -0.0693"/>
+    <axis rpy="0 0 0" xyz="1 0 0"/>
+  </joint>
+  <xacro:imu_sensor/>
+  <xacro:laser_sensor
+    update_rate="5"
+    ray_count="360"
+    min_angle="0"
+    max_angle="6.28"
+    min_range="0.12"
+    max_range="8.0"
+    topic_name="scan"
+    pos_x="0.27"
+    pos_y="0"
+    pos_z="0.188"
+  />
 </robot>

File: urdf/l1br_control.xacro (robot description, xacro)
@@ -1,4 +1,4 @@
 <?xml version="1.0" ?>
-<robot name="rocket" xmlns:xacro="http://ros.org/wiki/xacro">
+<robot name="l1br" xmlns:xacro="http://ros.org/wiki/xacro">
     <ros2_control name="GazeboSystem" type="system">
         <hardware>
@@ -24,5 +24,5 @@
     <gazebo>
         <plugin name="gazebo_ros2_control" filename="libgazebo_ros2_control.so">
-            <parameters>$(find rocket)/config/rocket_control.yaml</parameters>
+            <parameters>$(find l1br)/config/l1br_control.yaml</parameters>
         </plugin>
     </gazebo>

Commit message: xacrei rs

File: urdf/l1br.urdf.xacro (robot description, xacro)
@@ -5,300 +5,10 @@
   <xacro:include filename="sensors/imu_sensor.urdf.xacro" />
   <xacro:include filename="sensors/laser_sensor.urdf.xacro" />
-  <!--=========================== PLUGINS ===========================-->
-  <!-- <xacro:include filename="$(find l1br)/urdf/l1br.gazebo.xacro" /> -->
-  <!-- ****************** ROBOT CONSTANTS *******************************  -->
-  <!-- Define the size of the robot's main base_link in meters -->
-  <xacro:property name="base_width" value="0.47"/>
-  <xacro:property name="base_length" value="0.77"/>
-  <xacro:property name="base_height" value="0.13"/>
-  <!-- Define the shape of the robot's two wheels in meters -->
-  <xacro:property name="wheel_radius" value="0.0675"/>
-  <xacro:property name="wheel_width" value="0.04"/>
-  <!-- Define the shape of the robot's tray in meters -->
-  <xacro:property name="tray_radius" value="0.2"/>
-  <xacro:property name="tray_width" value="0.041"/>
-  <!-- Define the shape of the robot's four caster wheels in meters -->
-  <xacro:property name="caster_wheel_radius" value="0.01"/>
-  <!-- Colors -->
-  <material name="black">
-      <color rgba="0.0 0.0 0.0 1.0"/>
-  </material>
-  <!-- ********************** ROBOT BASE *********************************  -->
-  <link name="base_footprint">
-    </link>
-    <gazebo reference="base_link">
-      <mu1 value="0.3" />
-      <mu2 value="0.3" />
-      <kp value="1000000.0" />
-      <kd value="100" />
-      <fdir1 value="0 0 0" />
-    </gazebo>
-    <joint name="base_joint" type="fixed">
-      <parent link="base_link"/>
-      <child link="base_footprint" />
-      <origin xyz="0.0 0.0 -0.0793" rpy="0 0 3.14"/>
-    </joint>
-    <link name="base_link">
-      <visual>
-        <origin xyz="0  0  0" rpy="0 0 0"/>
-        <geometry>
-          <mesh filename="file:///$(find l1br)/meshes/EST_estrutura_m3.dae" />
-        </geometry>
-      </visual>
-      <collision>
-          <origin rpy="0  0  0" xyz="0  0  0.01" />
-          <geometry>
-              <box size="${base_length} ${base_width} ${base_height}"/>
-          </geometry>
-      </collision>
-      <inertial>
-          <origin xyz="0  0  0.0" rpy="0 0 1.57"/>
-          <mass value="2.4"/>
-          <inertia ixx="0.12196" ixy="0.0" ixz="0.0"
-                iyy="0.04756" iyz="0.0"
-                izz="0.16276" />
-      </inertial>
-    </link>
-  <!-- *********************** DRIVE WHEELS ******************************  -->
-    <gazebo reference="left_wheel">
-      <mu1>1.0</mu1>
-      <mu2>1.0</mu2>
-      <kp>1000000.0</kp>
-      <kd>100.0</kd>
-    </gazebo>
-    <link name="left_wheel">
-      <visual name="left_wheel_visual">
-        <origin xyz="0 0 0" rpy="0 0 0"/>
-        <geometry>
-            <mesh filename="file:///$(find l1br)/meshes/M_rodatrativa.dae" scale="1 1 1"/>
-        </geometry>
-      </visual>
-      <collision name="left_wheel_collision">
-        <origin xyz="0 0 0" rpy="0 1.57 0"/>
-        <geometry>
-          <cylinder length="${wheel_width}" radius="${wheel_radius}"/>
-        </geometry>
-      </collision>
-      <inertial>
-        <origin rpy="0 1.57 0" xyz="0 0 0" />
-        <mass value="1"/>
-        <inertia ixx="${(2/5) * 1 * (wheel_radius * wheel_radius)}" ixy="0" ixz="0"
-                iyy="${(2/5) * 1 * (wheel_radius * wheel_radius)}" iyz="0"
-                izz="${(2/5) * 1 * (wheel_radius * wheel_radius)}" />
-      </inertial>
-    </link>
-    <joint name="joint_left_wheel" type="continuous">
-            <parent link="base_link" />
-            <child link="left_wheel" />
-            <origin rpy="0 0 1.57" xyz=" 0 0.296755 -0.0118" />
-            <axis rpy="0 0 0" xyz="1 0 0"/>
-    </joint>
-    <gazebo reference="right_wheel">
-      <!-- <selfCollide>false</selfCollide> -->
-      <mu1>1.0</mu1>
-      <mu2>1.0</mu2>
-      <kp>1000000.0</kp>
-      <kd>100.0</kd>
-      <!-- <maxVel>1.0</maxVel> -->
-      <!-- <fdir1 value="0 0 0" /> -->
-    </gazebo>
-    <link name="right_wheel">
-      <visual name="right_wheel_visual">
-        <origin xyz="0 0 0" rpy="0 0 0"/>
-        <geometry>
-            <mesh filename="file:///$(find l1br)/meshes/M_rodatrativa.dae" scale="1 1 1"/>
-        </geometry>
-      </visual>
-      <collision name="right_wheel_collision">
-        <origin xyz="0 0 0" rpy="0 1.57 0"/>
-        <geometry>
-          <cylinder length="${wheel_width}" radius="${wheel_radius}"/>
-        </geometry>
-      </collision>
-      <inertial>
-        <origin rpy="0 1.57 0" xyz="0 0 0" />
-        <mass value="1"/>
-        <inertia ixx="${(2/5) * 1 * (wheel_radius * wheel_radius)}" ixy="0" ixz="0"
-                iyy="${(2/5) * 1 * (wheel_radius * wheel_radius)}" iyz="0"
-                izz="${(2/5) * 1 * (wheel_radius * wheel_radius)}" />
-      </inertial>
-    </link>
-    <joint name="joint_right_wheel" type="continuous">
-            <parent link="base_link" />
-            <child link="right_wheel" />
-            <origin rpy="0 0 1.57" xyz="0 -0.296395 -0.0118" />
-            <axis rpy="0 0 0" xyz="1 0 0"/>
-    </joint>
-  <!-- *********************** TRAY ******************************  -->
-  <link name="tray">
-      <visual name="tray_visual">
-        <origin xyz="0 0 0.0118" rpy="0 0 0"/>
-        <geometry>
-            <mesh filename="file:///$(find l1br)/meshes/ELV_conjuntocompleto.dae" scale="1 1 1"/>
-        </geometry>
-      </visual>
-      <collision name="tray_collision">
-        <origin xyz="0 -0.015047 0.1" rpy="0 0 0"/>
-        <geometry>
-          <cylinder length="${tray_width}" radius="${tray_radius}"/>
-        </geometry>
-      </collision>
-      <inertial>
-        <mass value="0.5" />
-        <origin rpy="0 0 0" xyz="0 0 0" />
-        <inertia ixx="0.0" ixy="0.0" ixz="0.0"
-                iyy="0.0" iyz="0.0"
-                izz="0.0" />
-      </inertial>
-  </link>
-  <joint name="joint_tray" type="fixed">
-            <parent link="base_link" />
-            <child link="tray" />
-            <origin rpy="0 0 0" xyz="0 0.015047 0" />
-  </joint>
-  <!-- *********************** CASTER WHEELS ******************************  -->
-  <gazebo reference="back_left_caster_wheel">
-      <selfCollide>false</selfCollide>
-      <mu1 value="0.09" />
-      <mu2 value="0.09" />
-      <kp value="10000000.0" />
-      <kd value="10000" />
-  </gazebo>
-  <link name="back_left_caster_wheel">
-    <visual name="back_left_caster_wheel_visual">
-      <origin xyz="0 0 0" rpy="0 0 0"/>
-      <geometry>
-        <sphere radius="${caster_wheel_radius}"/>
-      </geometry>
-      <material name="black"/>
-    </visual>
-    <collision name="back_left_caster_wheel_collision">
-      <origin xyz="0 0 0" rpy="0 0 0"/>
-      <geometry>
-        <sphere radius="0.01"/>
-      </geometry>
-    </collision>
-    <inertial>
-      <origin xyz="0 0 0" rpy="0 0 0"/>
-      <mass value="0.005"/>
-      <inertia ixx="${(2/5) * 0.005 * (caster_wheel_radius * caster_wheel_radius)}" ixy="0" ixz="0"
-              iyy="${(2/5) * 0.005 * (caster_wheel_radius * caster_wheel_radius)}" iyz="0"
-              izz="${(2/5) * 0.005 * (caster_wheel_radius * caster_wheel_radius)}" />
-    </inertial>
-  </link>
-  <joint name="joint_back_left_caster_wheel" type="continuous">
-    <parent link="base_link"/>
-    <child link="back_left_caster_wheel"/>
-    <origin rpy="-1.57 0 0" xyz="0.32 0.07 -0.0693"/>
-    <axis rpy="0 0 0" xyz="1 0 0"/>
-  </joint>
-  <gazebo reference="back_right_caster_wheel">
-      <selfCollide>false</selfCollide>
-      <mu1 value="0.09" />
-      <mu2 value="0.09" />
-      <kp value="10000000.0" />
-      <kd value="10000" />
-      <!-- <fdir1 value="0 0 0" /> -->
-  </gazebo>
-  <link name="back_right_caster_wheel">
-    <visual name="back_right_caster_wheel_visual">
-      <origin xyz="0 0 0" rpy="0 0 0"/>
-      <geometry>
-        <sphere radius="${caster_wheel_radius}"/>
-      </geometry>
-      <material name="black"/>
-    </visual>
-    <collision name="back_right_caster_wheel_collision">
-      <origin xyz="0 0 0" rpy="0 0 0"/>
-      <geometry>
-        <sphere radius="0.01"/>
-      </geometry>
-    </collision>
-    <inertial>
-      <origin xyz="0 0 0" rpy="0 0 0"/>
-      <mass value="0.005"/>
-      <inertia ixx="${(2/5) * 0.005 * (caster_wheel_radius * caster_wheel_radius)}" ixy="0" ixz="0"
-              iyy="${(2/5) * 0.005 * (caster_wheel_radius * caster_wheel_radius)}" iyz="0"
-              izz="${(2/5) * 0.005 * (caster_wheel_radius * caster_wheel_radius)}" />
-    </inertial>
-  </link>
-  <joint name="joint_back_right_caster_wheel" type="continuous">
-    <parent link="base_link"/>
-    <child link="back_right_caster_wheel"/>
-    <origin rpy="-1.57 0 0" xyz="0.32 -0.07 -0.0693"/>
-    <axis rpy="0 0 0" xyz="1 0 0"/>
-  </joint>
-  <gazebo reference="front_left_caster_wheel">
-      <selfCollide>false</selfCollide>
-      <mu1 value="0.09" />
-      <mu2 value="0.09" />
-      <kp value="10000000.0" />
-      <kd value="10000" />
-      <!-- <fdir1 value="0 0 0" /> -->
-  </gazebo>
-  <link name="front_left_caster_wheel">
-    <visual name="front_left_caster_wheel_visual">
-      <origin xyz="0 0 0" rpy="0 0 0"/>
-      <geometry>
-        <sphere radius="${caster_wheel_radius}"/>
-      </geometry>
-      <material name="black"/>
-    </visual>
-    <collision name="front_left_caster_wheel_collision">
-      <origin xyz="0 0 0" rpy="0 0 0"/>
-      <geometry>
-        <sphere radius="0.01"/>
-      </geometry>
-    </collision>
-    <inertial>
-      <origin xyz="0 0 0" rpy="0 0 0"/>
-      <mass value="0.005"/>
-      <inertia ixx="${(2/5) * 0.005 * (caster_wheel_radius * caster_wheel_radius)}" ixy="0" ixz="0"
-              iyy="${(2/5) * 0.005 * (caster_wheel_radius * caster_wheel_radius)}" iyz="0"
-              izz="${(2/5) * 0.005 * (caster_wheel_radius * caster_wheel_radius)}" />
-    </inertial>
-  </link>
-  <joint name="joint_front_left_caster_wheel" type="continuous">
-    <parent link="base_link"/>
-    <child link="front_left_caster_wheel"/>
-    <origin rpy="-1.57 0 0" xyz="-0.32 0.07 -0.0693"/>
-    <axis rpy="0 0 0" xyz="1 0 0"/>
-  </joint>
-  <gazebo reference="front_right_caster_wheel">
-      <selfCollide>false</selfCollide>
-      <mu1 value="0.09" />
-      <mu2 value="0.09" />
-      <kp value="10000000.0" />
-      <kd value="10000" />
-      <!-- <fdir1 value="0 0 0" /> -->
-  </gazebo>
-  <link name="front_right_caster_wheel">
-    <visual name="front_right_caster_wheel_visual">
-      <origin xyz="0 0 0" rpy="0 0 0"/>
-      <geometry>
-        <sphere radius="${caster_wheel_radius}"/>
-      </geometry>
-      <material name="black"/>
-    </visual>
-    <collision name="front_right_caster_wheel_collision">
-      <origin xyz="0 0 0" rpy="0 0 0"/>
-      <geometry>
-        <sphere radius="0.01"/>
-      </geometry>
-    </collision>
-    <inertial>
-      <origin xyz="0 0 0" rpy="0 0 0"/>
-      <mass value="0.005"/>
-      <inertia ixx="${(2/5) * 0.005 * (caster_wheel_radius * caster_wheel_radius)}" ixy="0" ixz="0"
-              iyy="${(2/5) * 0.005 * (caster_wheel_radius * caster_wheel_radius)}" iyz="0"
-              izz="${(2/5) * 0.005 * (caster_wheel_radius * caster_wheel_radius)}" />
-    </inertial>
-  </link>
-  <joint name="joint_front_right_caster_wheel" type="continuous">
-    <parent link="base_link"/>
-    <child link="front_right_caster_wheel"/>
-    <origin rpy="-1.57 0 0" xyz="-0.32 -0.07 -0.0693"/>
-    <axis rpy="0 0 0" xyz="1 0 0"/>
-  </joint>
+  <!-- =========================== ROBOT ===========================  -->
+  <xacro:include filename="robot_parts/traction_wheel.xacro" />
+  <xacro:include filename="robot_parts/caster_wheel.xacro" />
+  <xacro:include filename="robot_parts/robot_base.xacro" />
+  <xacro:include filename="robot_parts/tray.xacro" />
+  <xacro:tray/>
   <xacro:imu_sensor/>
   <xacro:laser_sensor

File: urdf/sensors/laser_sensor.urdf.xacro (robot description, xacro)
@@ -47,5 +47,5 @@
                 <update_rate>${update_rate}</update_rate>
                 <pose>0 0 0 0 0 0</pose>
-                <visualize>false</visualize>
+                <visualize>true</visualize>
                 <ray>
                     <scan>
