Commit message: tenho q ajeitar o pistao

File: urdf/l1br.urdf.xacro (robot description, xacro)
@@ -10,4 +10,5 @@
   <xacro:include filename="robot_parts/robot_base.xacro" />
   <xacro:include filename="robot_parts/tray.xacro" />
+  <xacro:include filename="robot_parts/piston.xacro" />
   <xacro:tray/>
   <xacro:imu_sensor/>

File: urdf/robot_parts/caster_wheel.xacro (robot description, xacro)
@@ -3,4 +3,5 @@
     <!-- Define the shape of the robot's four caster wheels in meters -->
     <xacro:property name="caster_wheel_radius" value="0.01"/>
+    <xacro:property name="caster_wheel_mass" value="0.005"/>
     <xacro:macro name="caster_wheel" params="prefix pos_X pos_Y pos_Z pos_r pos_p pos_y">
         <joint name="joint_${prefix}" type="continuous">
@@ -19,9 +20,9 @@
         <link name="${prefix}">
             <inertial>
-                <mass value="0.005" />
+                <mass value="${caster_wheel_mass}" />
                 <origin rpy="0 0 0" xyz="0 0 0" />
-                <inertia ixx="${(2/5) * 0.005 * (caster_wheel_radius * caster_wheel_radius)}" ixy="0" ixz="0"
-                         iyy="${(2/5) * 0.005 * (caster_wheel_radius * caster_wheel_radius)}" iyz="0"
-                         izz="${(2/5) * 0.005 * (caster_wheel_radius * caster_wheel_radius)}" />
+                <inertia ixx="${(2/5) * caster_wheel_mass * (caster_wheel_radius * caster_wheel_radius)}" ixy="0" ixz="0"
+                         iyy="${(2/5) * caster_wheel_mass * (caster_wheel_radius * caster_wheel_radius)}" iyz="0"
+                         izz="${(2/5) * caster_wheel_mass * (caster_wheel_radius * caster_wheel_radius)}" />
             </inertial>
             <collision name="${prefix}_collision">

File: urdf/robot_parts/robot_base.xacro (robot description, xacro)
@@ -5,4 +5,5 @@
     <xacro:property name="base_length" value="0.77"/>
     <xacro:property name="base_height" value="0.13"/>
+    <xacro:property name="base_mass" value="2.4"/>
     <xacro:macro name="base" params="base_link">
         <link name="base_footprint">
@@ -35,5 +36,5 @@
         <inertial>
             <origin xyz="0  0  0.0" rpy="0 0 1.57"/>
-            <mass value="2.4"/>
+            <mass value="${base_mass}"/>
             <inertia ixx="0.12196" ixy="0.0" ixz="0.0"
                     iyy="0.04756" iyz="0.0"

File: urdf/robot_parts/traction_wheel.xacro (robot description, xacro)
@@ -4,4 +4,5 @@
     <xacro:property name="wheel_radius" value="0.0675"/>
     <xacro:property name="wheel_width" value="0.04"/>
+    <xacro:property name="wheel_mass" value="1"/>
     <xacro:macro name="traction_wheel" params="prefix pos_X pos_Y pos_Z pos_r pos_p pos_y">
         <joint name="joint_${prefix}" type="continuous">
@@ -20,9 +21,9 @@
         <link name="${prefix}">
             <inertial>
-                <mass value="1" />
+                <mass value="${wheel_mass}" />
                 <origin rpy="0 1.57 0" xyz="0 0 0" />
-                <inertia ixx="${(2/5) * 1 * (wheel_radius * wheel_radius)}" ixy="0" ixz="0"
-                         iyy="${(2/5) * 1 * (wheel_radius * wheel_radius)}" iyz="0"
-                         izz="${(2/5) * 1 * (wheel_radius * wheel_radius)}" />
+                <inertia ixx="${(2/5) * wheel_mass * (wheel_radius * wheel_radius)}" ixy="0" ixz="0"
+                         iyy="${(2/5) * wheel_mass * (wheel_radius * wheel_radius)}" iyz="0"
+                         izz="${(2/5) * wheel_mass * (wheel_radius * wheel_radius)}" />
             </inertial>
             <collision name="${prefix}_collision">

File: urdf/robot_parts/tray.xacro (robot description, xacro)
@@ -21,13 +21,21 @@
             <mass value="0.5" />
             <origin rpy="0 0 0" xyz="0 0 0" />
-            <inertia ixx="0.0" ixy="0.0" ixz="0.0"
-                    iyy="0.0" iyz="0.0"
-                    izz="0.0" />
+            <inertia ixx="${(2/5) * 0.5 * (tray_radius * tray_radius)}" ixy="0.0" ixz="0.0"
+                    iyy="${(2/5) * 0.5 * (tray_radius * tray_radius)}" iyz="0.0"
+                    izz="${(2/5) * 0.5 * (tray_radius * tray_radius)}" />
         </inertial>
         </link>
-        <joint name="joint_tray" type="fixed">
-                <parent link="base_link" />
+        <!-- <joint name="joint_prismatic_tray" type="prismatic"> -->
+                <!-- <parent link="base_link" /> -->
+                <!-- <child link="tray" /> -->
+                <!-- <origin rpy="0 0 0" xyz="0 0.015047 0" /> -->
+                <!-- <axis xyz="0 0 1"/> -->
+                <!-- <limit effort="1000.0" lower="0" upper="0.3" velocity="0.5"/> -->
+        <!-- </joint> -->
+        <joint name="joint_tray" type="continuous">
+                <parent link="piston" />
                 <child link="tray" />
-                <origin rpy="0 0 0" xyz="0 0.015047 0" />
+                <origin rpy="0 0 0" xyz="0 0 0" />
+                <axis xyz="0 0 1"/>
         </joint>
     </xacro:macro>

Commit message: joints colocados

File: urdf/l1br.urdf.xacro (robot description, xacro)
@@ -10,6 +10,7 @@
   <xacro:include filename="robot_parts/robot_base.xacro" />
   <xacro:include filename="robot_parts/tray.xacro" />
+  <xacro:tray/>
   <xacro:include filename="robot_parts/piston.xacro" />
-  <xacro:tray/>
+  <xacro:piston/>
   <xacro:imu_sensor/>
   <xacro:laser_sensor

File: urdf/robot_parts/piston.xacro (robot description, xacro)
@@ -1,8 +1,15 @@
 <?xml version="1.0"?>
 <robot xmlns:xacro="http://www.ros.org/wiki/xacro">
-    <xacro:property name="piston_width" value="0.1"/>
-    <xacro:property name="piston_radius" value="0.2"/>
+    <xacro:property name="piston_width" value="0.01"/>
+    <xacro:property name="piston_radius" value="0.05"/>
     <xacro:property name="piston_mass" value="0.2"/>
     <xacro:macro name="piston">
+        <gazebo reference="piston">
+            <selfCollide>false</selfCollide>
+            <mu1>0.09</mu1>
+            <mu2>0.09</mu2>
+            <kp>10000000.0</kp>
+            <kd>10000.0</kd>
+        </gazebo>
         <link name="piston">
             <visual name="piston_visual">
@@ -29,5 +36,5 @@
                 <parent link="base_link" />
                 <child link="piston" />
-                <origin rpy="0 0 0" xyz="0 0.015047 0" />
+                <origin rpy="0 0 0" xyz="0 0 0.09" />
                 <axis xyz="0 0 1"/>
                 <limit effort="1000.0" lower="0" upper="0.3" velocity="0.5"/>

File: urdf/robot_parts/tray.xacro (robot description, xacro)
@@ -36,5 +36,5 @@
                 <parent link="piston" />
                 <child link="tray" />
-                <origin rpy="0 0 0" xyz="0 0 0" />
+                <origin rpy="0 0 0" xyz="0 0 -0.06" />
                 <axis xyz="0 0 1"/>
         </joint>
