Commit message: pistão 10/10

File: urdf/robot_parts/piston.xacro (robot description, xacro)
@@ -1,5 +1,5 @@
 <?xml version="1.0"?>
 <robot xmlns:xacro="http://www.ros.org/wiki/xacro">
-    <xacro:property name="piston_cylinder_width" value="0.13"/>
+    <xacro:property name="piston_cylinder_width" value="0.15"/>
     <xacro:property name="piston_cylinder_radius" value="0.015"/>
     <xacro:property name="piston_cylinder_mass" value="0.2"/>
@@ -41,5 +41,5 @@
                 <origin rpy="0 0 0" xyz="0 0 0.02" />
                 <axis xyz="0 0 1"/>
-                <limit effort="1000.0" lower="0" upper="0.1" velocity="0.5"/>
+                <limit effort="1000.0" lower="0" upper="0.12" velocity="0.5"/>
         </joint>
         <gazebo reference="piston_base">
@@ -74,5 +74,5 @@
                 <parent link="piston_cylinder" />
                 <child link="piston_base" />
-                <origin rpy="0 0 0" xyz="0 0 0.07" />
+                <origin rpy="0 0 0" xyz="0 0 0.08" />
         </joint>
     </xacro:macro>

Commit message: agora foi

File: urdf/robot_parts/piston.xacro (robot description, xacro)
@@ -1,5 +1,5 @@
 <?xml version="1.0"?>
 <robot xmlns:xacro="http://www.ros.org/wiki/xacro">
-    <xacro:property name="piston_cylinder_width" value="0.15"/>
+    <xacro:property name="piston_cylinder_width" value="0.19"/>
     <xacro:property name="piston_cylinder_radius" value="0.015"/>
     <xacro:property name="piston_cylinder_mass" value="0.2"/>
@@ -39,7 +39,7 @@
                 <parent link="base_link" />
                 <child link="piston_cylinder" />
-                <origin rpy="0 0 0" xyz="0 0 0.02" />
+                <origin rpy="0 0 0" xyz="0 0 0.03" />
                 <axis xyz="0 0 1"/>
-                <limit effort="1000.0" lower="0" upper="0.12" velocity="0.5"/>
+                <limit effort="1000.0" lower="0" upper="0.13" velocity="0.5"/>
         </joint>
         <gazebo reference="piston_base">
@@ -74,5 +74,5 @@
                 <parent link="piston_cylinder" />
                 <child link="piston_base" />
-                <origin rpy="0 0 0" xyz="0 0 0.08" />
+                <origin rpy="0 0 0" xyz="0 0 0.1" />
         </joint>
     </xacro:macro>
