Commit message: ideia do pistão feita

File: urdf/robot_parts/caster_wheel.xacro (robot description, xacro)
@@ -3,4 +3,5 @@
     <!-- Define the shape of the robot's four caster wheels in meters -->
     <xacro:property name="caster_wheel_radius" value="0.01"/>
+    <xacro:property name="caster_wheel_radius_visual" value="0.001"/>
     <xacro:property name="caster_wheel_mass" value="0.005"/>
     <xacro:macro name="caster_wheel" params="prefix pos_X pos_Y pos_Z pos_r pos_p pos_y">
@@ -35,5 +36,5 @@
                 <origin rpy="0 0 0" xyz="0 0 0" />
                 <geometry>
-                    <sphere radius="${caster_wheel_radius}"/>
+                    <sphere radius="${caster_wheel_radius_visual}"/>
                 </geometry>
             </visual>

File: urdf/robot_parts/piston.xacro (robot description, xacro)
@@ -1,9 +1,12 @@
 <?xml version="1.0"?>
 <robot xmlns:xacro="http://www.ros.org/wiki/xacro">
-    <xacro:property name="piston_width" value="0.01"/>
-    <xacro:property name="piston_radius" value="0.05"/>
-    <xacro:property name="piston_mass" value="0.2"/>
+    <xacro:property name="piston_cylinder_width" value="0.13"/>
+    <xacro:property name="piston_cylinder_radius" value="0.015"/>
+    <xacro:property name="piston_cylinder_mass" value="0.2"/>
+    <xacro:property name="piston_base_width" value="0.01"/>
+    <xacro:property name="piston_base_radius" value="0.08"/>
+    <xacro:property name="piston_base_mass" value="0.2"/>
     <xacro:macro name="piston">
-        <gazebo reference="piston">
+        <gazebo reference="piston_cylinder">
             <selfCollide>false</selfCollide>
             <mu1>0.09</mu1>
@@ -12,31 +15,64 @@
             <kd>10000.0</kd>
         </gazebo>
-        <link name="piston">
-            <visual name="piston_visual">
+        <link name="piston_cylinder">
+            <visual name="piston_cylinder_visual">
                 <origin xyz="0 0 0" rpy="0 0 0"/>
                 <geometry>
-                    <cylinder length="${piston_width}" radius="${piston_radius}"/>
+                    <cylinder length="${piston_cylinder_width}" radius="${piston_cylinder_radius}"/>
                 </geometry>
             </visual>
-            <collision name="piston_collision">
+            <!-- <collision name="piston_cylinder_collision"> -->
+                <!-- <origin xyz="0 0 0" rpy="0 0 0"/> -->
+                <!-- <geometry> -->
+                    <!-- <cylinder length="${piston_cylinder_width}" radius="${piston_cylinder_radius}"/> -->
+                <!-- </geometry> -->
+            <!-- </collision> -->
+            <inertial>
+                <mass value="${piston_cylinder_mass}" />
+                <origin rpy="0 0 0" xyz="0 0 0" />
+                <inertia ixx="${(2/5) * piston_cylinder_mass * (piston_cylinder_radius * piston_cylinder_radius)}" ixy="0.0" ixz="0.0"
+                        iyy="${(2/5) * piston_cylinder_mass * (piston_cylinder_radius * piston_cylinder_radius)}" iyz="0.0"
+                        izz="${(2/5) * piston_cylinder_mass * (piston_cylinder_radius * piston_cylinder_radius)}" />
+            </inertial>
+        </link>
+        <joint name="joint_piston_cylinder" type="prismatic">
+                <parent link="base_link" />
+                <child link="piston_cylinder" />
+                <origin rpy="0 0 0" xyz="0 0 0.02" />
+                <axis xyz="0 0 1"/>
+                <limit effort="1000.0" lower="0" upper="0.1" velocity="0.5"/>
+        </joint>
+        <gazebo reference="piston_base">
+            <selfCollide>false</selfCollide>
+            <mu1>0.09</mu1>
+            <mu2>0.09</mu2>
+            <kp>10000000.0</kp>
+            <kd>10000.0</kd>
+        </gazebo>
+        <link name="piston_base">
+            <visual name="piston_base_visual">
                 <origin xyz="0 0 0" rpy="0 0 0"/>
                 <geometry>
-                    <cylinder length="${piston_width}" radius="${piston_radius}"/>
+                    <cylinder length="${piston_base_width}" radius="${piston_base_radius}"/>
+                </geometry>
+            </visual>
+            <collision name="piston_base_collision">
+                <origin xyz="0 0 0" rpy="0 0 0"/>
+                <geometry>
+                    <cylinder length="${piston_base_width}" radius="${piston_base_radius}"/>
                 </geometry>
             </collision>
             <inertial>
-                <mass value="${piston_mass}" />
+                <mass value="${piston_base_mass}" />
                 <origin rpy="0 0 0" xyz="0 0 0" />
-                <inertia ixx="${(2/5) * piston_mass * (piston_radius * piston_radius)}" ixy="0.0" ixz="0.0"
-                        iyy="${(2/5) * piston_mass * (piston_radius * piston_radius)}" iyz="0.0"
-                        izz="${(2/5) * piston_mass * (piston_radius * piston_radius)}" />
+                <inertia ixx="${(2/5) * piston_base_mass * (piston_base_radius * piston_base_radius)}" ixy="0.0" ixz="0.0"
+                        iyy="${(2/5) * piston_base_mass * (piston_base_radius * piston_base_radius)}" iyz="0.0"
+                        izz="${(2/5) * piston_base_mass * (piston_base_radius * piston_base_radius)}" />
             </inertial>
         </link>
-        <joint name="joint_piston" type="prismatic">
-                <parent link="base_link" />
-                <child link="piston" />
-                <origin rpy="0 0 0" xyz="0 0 0.09" />
-                <axis xyz="0 0 1"/>
-                <limit effort="1000.0" lower="0" upper="0.3" velocity="0.5"/>
+        <joint name="joint_base_cylinder" type="fixed">
+                <parent link="piston_cylinder" />
+                <child link="piston_base" />
+                <origin rpy="0 0 0" xyz="0 0 0.07" />
         </joint>
     </xacro:macro>

File: urdf/robot_parts/tray.xacro (robot description, xacro)
@@ -3,5 +3,5 @@
     <!-- Define the shape of the robot's tray in meters -->
     <xacro:property name="tray_radius" value="0.2"/>
-    <xacro:property name="tray_width" value="0.041"/>
+    <xacro:property name="tray_width" value="0.03"/>
     <xacro:macro name="tray">
         <link name="tray">
@@ -13,5 +13,5 @@
         </visual>
         <collision name="tray_collision">
-            <origin xyz="0 -0.015047 0.1" rpy="0 0 0"/>
+            <origin xyz="0 0 0.105" rpy="0 0 0"/>
             <geometry>
             <cylinder length="${tray_width}" radius="${tray_radius}"/>
@@ -34,7 +34,7 @@
         <!-- </joint> -->
         <joint name="joint_tray" type="continuous">
-                <parent link="piston" />
+                <parent link="piston_base" />
                 <child link="tray" />
-                <origin rpy="0 0 0" xyz="0 0 -0.06" />
+                <origin rpy="0 0 0" xyz="0 0 -0.08" />
                 <axis xyz="0 0 1"/>
         </joint>

Commit message: lembro oq eu fiz nao

File: urdf/robot_parts/caster_wheel.xacro (robot description, xacro)
@@ -14,6 +14,6 @@
         <gazebo reference="${prefix}">
             <selfCollide>false</selfCollide>
-            <mu1>0.09</mu1>
-            <mu2>0.09</mu2>
+            <mu1>0.2</mu1>
+            <mu2>0.2</mu2>
             <kp>10000000.0</kp>
             <kd>10000.0</kd>
@@ -41,7 +41,7 @@
         </link>
     </xacro:macro>
-    <xacro:caster_wheel prefix="back_left_caster_wheel" pos_X="0.32" pos_Y="0.07" pos_Z="-0.0693" pos_r="-1.57" pos_p="0" pos_y="0" />
-    <xacro:caster_wheel prefix="back_right_caster_wheel" pos_X="0.32" pos_Y="-0.07" pos_Z="-0.0693" pos_r="-1.57" pos_p="0" pos_y="0" />
-    <xacro:caster_wheel prefix="front_left_caster_wheel" pos_X="-0.32" pos_Y="0.07" pos_Z="-0.0693" pos_r="-1.57" pos_p="0" pos_y="0" />
-    <xacro:caster_wheel prefix="front_right_caster_wheel" pos_X="-0.32" pos_Y="-0.07" pos_Z="-0.0693" pos_r="-1.57" pos_p="0" pos_y="0" />
+    <xacro:caster_wheel prefix="back_left_caster_wheel" pos_X="0.32" pos_Y="0.07" pos_Z="-0.092" pos_r="-1.57" pos_p="0" pos_y="0" />
+    <xacro:caster_wheel prefix="back_right_caster_wheel" pos_X="0.32" pos_Y="-0.07" pos_Z="-0.092" pos_r="-1.57" pos_p="0" pos_y="0" />
+    <xacro:caster_wheel prefix="front_left_caster_wheel" pos_X="-0.32" pos_Y="0.07" pos_Z="-0.092" pos_r="-1.57" pos_p="0" pos_y="0" />
+    <xacro:caster_wheel prefix="front_right_caster_wheel" pos_X="-0.32" pos_Y="-0.07" pos_Z="-0.092" pos_r="-1.57" pos_p="0" pos_y="0" />
 </robot>

File: urdf/robot_parts/piston.xacro (robot description, xacro)
@@ -1,5 +1,5 @@
 <?xml version="1.0"?>
 <robot xmlns:xacro="http://www.ros.org/wiki/xacro">
-    <xacro:property name="piston_cylinder_width" value="0.19"/>
+    <xacro:property name="piston_cylinder_width" value="0.15"/>
     <xacro:property name="piston_cylinder_radius" value="0.015"/>
     <xacro:property name="piston_cylinder_mass" value="0.2"/>
@@ -10,6 +10,6 @@
         <gazebo reference="piston_cylinder">
             <selfCollide>false</selfCollide>
-            <mu1>0.09</mu1>
-            <mu2>0.09</mu2>
+            <mu1>0.1</mu1>
+            <mu2>0.1</mu2>
             <kp>10000000.0</kp>
             <kd>10000.0</kd>
@@ -21,4 +21,7 @@
                     <cylinder length="${piston_cylinder_width}" radius="${piston_cylinder_radius}"/>
                 </geometry>
+                <material name="grey">
+                    <color rgba="0.2 0.2 0.2 1.0"/>
+                </material>
             </visual>
             <!-- <collision name="piston_cylinder_collision"> -->
@@ -39,12 +42,12 @@
                 <parent link="base_link" />
                 <child link="piston_cylinder" />
-                <origin rpy="0 0 0" xyz="0 0 0.03" />
+                <origin rpy="0 0 0" xyz="0 0 0.02" />
                 <axis xyz="0 0 1"/>
-                <limit effort="1000.0" lower="0" upper="0.13" velocity="0.5"/>
+                <limit effort="1000.0" lower="0" upper="0.12" velocity="0.3"/>
         </joint>
         <gazebo reference="piston_base">
             <selfCollide>false</selfCollide>
-            <mu1>0.09</mu1>
-            <mu2>0.09</mu2>
+            <mu1>0.3</mu1>
+            <mu2>0.3</mu2>
             <kp>10000000.0</kp>
             <kd>10000.0</kd>
@@ -56,4 +59,7 @@
                     <cylinder length="${piston_base_width}" radius="${piston_base_radius}"/>
                 </geometry>
+                <material name="grey">
+                    <color rgba="0.2 0.2 0.2 1.0"/>
+                </material>
             </visual>
             <collision name="piston_base_collision">
@@ -74,5 +80,5 @@
                 <parent link="piston_cylinder" />
                 <child link="piston_base" />
-                <origin rpy="0 0 0" xyz="0 0 0.1" />
+                <origin rpy="0 0 0" xyz="0 0 0.08" />
         </joint>
     </xacro:macro>

File: urdf/robot_parts/traction_wheel.xacro (robot description, xacro)
@@ -14,6 +14,6 @@
         <gazebo reference="${prefix}">
             <selfCollide>false</selfCollide>
-            <mu1>1.0</mu1>
-            <mu2>1.0</mu2>
+            <mu1>1.5</mu1>
+            <mu2>1.5</mu2>
             <kp>1000000.0</kp>
             <kd>100.0</kd>

File: urdf/robot_parts/tray.xacro (robot description, xacro)
@@ -3,4 +3,5 @@
     <!-- Define the shape of the robot's tray in meters -->
     <xacro:property name="tray_radius" value="0.2"/>
+    <!-- antigo raio era 0.2 -->
     <xacro:property name="tray_width" value="0.03"/>
     <xacro:macro name="tray">
@@ -26,4 +27,12 @@
         </inertial>
         </link>
+        <gazebo reference="tray">
+            <selfCollide>true</selfCollide>
+            <mu1 value="1.5" />
+            <mu2 value="1.5" />
+            <kp value="10000000.0" />
+            <kd value="10000" />
+            <fdir1 value="0 0 0" />
+        </gazebo>
         <!-- <joint name="joint_prismatic_tray" type="prismatic"> -->
                 <!-- <parent link="base_link" /> -->
